File: electronics/moduleDriver.sch (KiCad schematic (older format))
At the start: 30 parts, among them J1 Screw_Terminal_01x03, U1 Mega2560Shield, U10 ULN2003AModule, U11 ULN2003AModule, U12 ULN2003AModule, U13 ULN2003AModule, U14 SSD1306_I2C, U15 INA219_Breakout, U2 ULN2003AModule, U3 ULN2003AModule, U4 ULN2003AModule, U5 ULN2003AModule, U6 ULN2003AModule, U7 ULN2003AModule, U8 ULN2003AModule, U9 ULN2003AModule

Commit message: More schematic progress
Parts:
- added U?: ST7789_IPS, symbol LCD:ST7789_IPS
Connections:
- net MOTOR_CLOCK is gone; now on net CLOCK: U?.11 (SRCLK), U?.11 (SRCLK), U?.11 (SRCLK), U?.11 (SRCLK), U?.11 (SRCLK)
- net SENSOR_CLOCK is gone; now on net CLOCK: U?.2 (CLK), U?.2 (CLK)
- net +3V3: now also U?.12 (3V3), U?.24 (3V3), U?.VCC
- net +5V: now also U?.13 (5V)
- net CLOCK: now also U?.18 (GPIO33)
- net GND: now also U?.1 (GND), U?.10 (GND), U?.11 (GND), U?.14 (GND), U?.2 (GND), U?.GND
- net MOTOR_DATA: now also U?.19 (GPIO32)
- net MOTOR_LATCH: now also U?.17 (GPIO25)
- net MOTOR_OE: now also U?.15 (GPIO27)
- net RX: now also U?.3 (GPIO21)
- net SCL: now also U?.21 (GPIO38)
- net SDA: now also U?.22 (GPIO37)
- net SENSOR_A: now also U1.D41
- net SENSOR_B: now also U1.D40
- net SENSOR_C: now also U1.D39
- net SENSOR_D: now also U1.D38
- net SENSOR_DATA: now also U?.20 (GPIO39)
- net SENSOR_E: now also U1.D19
- net SENSOR_F: now also U1.D18
- net SENSOR_G: now also U1.D17
- net SENSOR_H: now also U1.D16
- net SENSOR_I: now also U1.D15
- net SENSOR_J: now also U1.D14
- net SENSOR_K: now also U1.D2
- net SENSOR_L: now also U1.D3
- net SENSOR_LATCH: now also U?.16 (GPIO26)
- net TX: now also U?.4 (GPIO22)
- new net DISP_BLK: U?.BLK
- new net DISP_CLK: U?.SCL (SCL(CLK))
- new net DISP_CS: U?.CS
- new net DISP_DC: U?.DC
- new net DISP_MOSI: U?.SDA (SDA_(MOSI))
- new net DISP_RES: U?.RES
Other:
- moved on the sheet: U?
