File: electronics/moduleDriver/moduleDriver.sch (KiCad schematic (older format))
At the start: 114 parts, among them J1 Power In, J10 12V SENSE, J11 Motor A, J12 Motor E, J13 Motor I, J14 Motor B, J15 Motor F, J16 Motor J, J17 Motor C, J18 Motor G, J19 Motor K, J2 UART, J20 Motor D, J21 Motor H, J22 Motor L, J3 SENSOR, J4 IOVCC, J5 GND, J6 SR CHAIN IN, J7 SR CHAIN OUT, J8 RS485, J9 RS485, Q1 BSS138, Q2 BSS138, U1 Mega2560Shield, U10 ULN2003AModule, U11 INA219 Breakout Wide (blue), U12 ULN2003AModule, U13 ULN2003AModule, U14 ULN2003AModule, U15 ULN2003AModule, U16 LevelShifterModule, U17 RS485Module, U18 TTGO_TDisplay, U19 74HC244, U2 SSD1306_I2C, U20 74HC165, U21 74HC165, U22 ST7789_80x160, U23 D1_32, U24 74HC595, U25 74HC595, U26 74HC595, U27 74HC595, U28 74HC595, U29 74HC595, U3 ULN2003AModule, U30 ST7789_240x240, U31 INA219 Breakout Narrow (purpl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, U32 SP485, U33 INA219BxD, U34 TPL7407LA, U35 TPL7407LA, U36 TPL7407LA, U37 TPL7407LA, U38 TPL7407LA, U39 TPL7407LA, U4 ULN2003AModule, U40 TPL7407LA, U5 ULN2003AModule, U6 ULN2003AModule, U7 ULN2003AModule, U8 ULN2003AModule, U9 ULN2003AModule

Commit message: centralize libraries
Parts:
- U20, U21: symbol 74HC165:74HC165 -> 74HC165_2:74HC165
Changed lines of the file:
@@
 	7100 12700 7100 13000
 Connection ~ 7600 13000
-$Comp
-L 74HC165:74HC165 U21
-U 1 1 5FC6DACF
-P 4600 12400
-F 0 "U21" H 4700 13150 50  0000 C CNN
-F 1 "74HC165" H 4850 13050 50  0000 C CNN
-F 2 "Package_DIP:DIP-16_W7.62mm" H 5200 13600 50  0001 C CNN
-F 3 "DOCUMENTATION" H 5350 13500 50  0001 C CNN
-	1    4600 12400
-	1    0    0    -1
-$EndComp
 Text Label 5650 11900 2    50   ~ 0
 SENSOR_A
@@
 Wire Wire Line
 	3950 12350 4000 12350
-$Comp
-L 74HC165:74HC165 U20
-U 1 1 5FF4AE84
-P 2150 12400
-F 0 "U20" H 2250 13150 50  0000 C CNN
-F 1 "74HC165" H 2400 13050 50  0000 C CNN
-F 2 "Package_DIP:DIP-16_W7.62mm" H 2750 13600 50  0001 C CNN
-F 3 "DOCUMENTATION" H 2900 13500 50  0001 C CNN
-	1    2150 12400
-	1    0    0    -1
-$EndComp
 Text Label 3200 11900 2    50   ~ 0
 SENSOR_I
@@
 	1    0    0    -1
 $EndComp
-$Comp
-L LevelShifterModule:LevelShifterModule U16
-U 1 1 60E2A3B1
-P 14500 10600
-F 0 "U16" H 14500 11075 50  0000 C CNN
-F 1 "LevelShifterModule" H 14500 10984 50  0000 C CNN
-F 2 "LevelShifterModule:LevelShifterModule" H 14350 10650 50  0001 C CNN
-F 3 "" H 14350 10650 50  0001 C CNN
-	1    14500 10600
-	1    0    0    -1
-$EndComp
 Wire Wire Line
 	12400 8100 13350 8100
@@
 Connection ~ 6050 7200
 Wire Wire Line
-	7650 6750 7650 6850
-Wire Wire Line
 	7650 7200 8100 7200
+Wire Wire Line
+	7650 6750 7650 6850
 Connection ~ 7650 6850
 Wire Wire Line
 	7650 6850 7650 6950
-Connection ~ 7650 6950
 Wire Wire Line
 	7650 6950 7650 7200
+Connection ~ 7650 6950
 Connection ~ 8100 7200
+$Comp
+L LevelShifterModule:LevelShifterModule U16
+U 1 1 60E2A3B1
+P 14500 10600
+F 0 "U16" H 14500 11075 50  0000 C CNN
+F 1 "LevelShifterModule" H 14500 10984 50  0000 C CNN
+F 2 "LevelShifterModule:LevelShifterModule" H 14350 10650 50  0001 C CNN
+F 3 "" H 14350 10650 50  0001 C CNN
+	1    14500 10600
+	1    0    0    -1
+$EndComp
+$Comp
+L 74HC165_2:74HC165 U20
+U 1 1 5FF4AE84
+P 2150 12400
+F 0 "U20" H 2250 13150 50  0000 C CNN
+F 1 "74HC165" H 2400 13050 50  0000 C CNN
+F 2 "Package_DIP:DIP-16_W7.62mm" H 2750 13600 50  0001 C CNN
+F 3 "DOCUMENTATION" H 2900 13500 50  0001 C CNN
+	1    2150 12400
+	1    0    0    -1
+$EndComp
+$Comp
+L 74HC165_2:74HC165 U21
+U 1 1 5FC6DACF
+P 4600 12400
+F 0 "U21" H 4700 13150 50  0000 C CNN
+F 1 "74HC165" H 4850 13050 50  0000 C CNN
+F 2 "Package_DIP:DIP-16_W7.62mm" H 5200 13600 50  0001 C CNN
+F 3 "DOCUMENTATION" H 5350 13500 50  0001 C CNN
+	1    4600 12400
+	1    0    0    -1
+$EndComp
 $EndSCHEMATC

Commit message: Checkpoint
Parts:
- removed C17, C18, C19, C20, C21, C22: 0.1uF, symbol Device:C_Small
- removed J11: Motor A, JST_XH_Connectors:JST_XH_2-5mm_5pin, symbol Connector:Conn_01x05_Male
- removed J12: Motor E, JST_XH_Connectors:JST_XH_2-5mm_5pin, symbol Connector:Conn_01x05_Male
- removed J13: Motor I, JST_XH_Connectors:JST_XH_2-5mm_5pin, symbol Connector:Conn_01x05_Male
- removed J14: Motor B, JST_XH_Connectors:JST_XH_2-5mm_5pin, symbol Connector:Conn_01x05_Male
- removed J15: Motor F, JST_XH_Connectors:JST_XH_2-5mm_5pin, symbol Connector:Conn_01x05_Male
- removed J16: Motor J, JST_XH_Connectors:JST_XH_2-5mm_5pin, symbol Connector:Conn_01x05_Male
- removed J17: Motor C, JST_XH_Connectors:JST_XH_2-5mm_5pin, symbol Connector:Conn_01x05_Male
- removed J18: Motor G, JST_XH_Connectors:JST_XH_2-5mm_5pin, symbol Connector:Conn_01x05_Male
- removed J19: Motor K, JST_XH_Connectors:JST_XH_2-5mm_5pin, symbol Connector:Conn_01x05_Male
- removed J20: Motor D, JST_XH_Connectors:JST_XH_2-5mm_5pin, symbol Connector:Conn_01x05_Male
- removed J21: Motor H, JST_XH_Connectors:JST_XH_2-5mm_5pin, symbol Connector:Conn_01x05_Male
- removed J22: Motor L, JST_XH_Connectors:JST_XH_2-5mm_5pin, symbol Connector:Conn_01x05_Male
- removed J6: SR CHAIN IN, Connector_PinSocket_2.54mm:PinSocket_1x06_P2.54mm_Vertical, symbol Connector:Screw_Terminal_01x06
- removed J7: SR CHAIN OUT, Connector_PinSocket_2.54mm:PinSocket_1x06_P2.54mm_Vertical, symbol Connector:Screw_Terminal_01x06
- removed JP2: RX 3.3V, Jumper:SolderJumper-2_P1.3mm_Open_TrianglePad1.0x1.5mm, symbol Jumper:SolderJumper_2_Open
- removed JP3: TX 3.3V, Jumper:SolderJumper-2_P1.3mm_Open_TrianglePad1.0x1.5mm, symbol Jumper:SolderJumper_2_Open
- removed Q1, Q2: BSS138, Package_TO_SOT_SMD:SOT-23, symbol Transistor_FET:BSS138
- removed R1, R10, R11, R12, R2, R3, R4, R5, R6, R7, R8, R9: 47k, Resistor_THT:R_Axial_DIN0204_L3.6mm_D1.6mm_P1.90mm_Vertical, symbol Device:R_Small
- removed R13, R14, R15, R16: 10k, Resistor_SMD:R_0805_2012Metric_Pad1.15x1.40mm_HandSolder, symbol Device:R_Small
- removed U16: LevelShifterModule, LevelShifterModule:LevelShifterModule, symbol LevelShifterModule:LevelShifterModule
- removed U18: TTGO_TDisplay, ESP32:T-DISPLAY, symbol ESP32Modules:TTGO_TDisplay
- removed U19: 74HC244, Package_DIP:DIP-20_W7.62mm, symbol 74xx:74HC244
- removed U20, U21: 74HC165, Package_DIP:DIP-16_W7.62mm, symbol 74HC165_2:74HC165
- removed U22: ST7789_80x160, ST7789:ST7789_80x160, symbol LCD:ST7789_80x160
- removed U23: D1_32, ESP32:D1_32, symbol ESP32Modules:D1_32
- removed U24, U25, U26, U27, U28, U29: 74HC595, Package_DIP:DIP-16_W7.62mm, symbol 74xx:74HC595
- removed U30: ST7789_240x240, ST7789:ST7789_240x240, symbol LCD:ST7789_240x240
- removed U34, U35, U36, U37, U38, U39, U40: TPL7407LA, Package_SO:SOIC-16_3.9x9.9mm_P1.27mm, symbol Transistor_Array:ULN2003A
- added D1: SK6812_A, LED_SMD:LED_SK6812_PLCC4_5.0x5.0mm_P3.2mm, symbol LED:SK6812
- added D10: SK6812_J, LED_SMD:LED_SK6812_PLCC4_5.0x5.0mm_P3.2mm, symbol LED:SK6812
- added D11: SK6812_K, LED_SMD:LED_SK6812_PLCC4_5.0x5.0mm_P3.2mm, symbol LED:SK6812
- added D12: SK6812_L, LED_SMD:LED_SK6812_PLCC4_5.0x5.0mm_P3.2mm, symbol LED:SK6812
- added D2: SK6812_B, LED_SMD:LED_SK6812_PLCC4_5.0x5.0mm_P3.2mm, symbol LED:SK6812
- added D3: SK6812_C, LED_SMD:LED_SK6812_PLCC4_5.0x5.0mm_P3.2mm, symbol LED:SK6812
- added D4: SK6812_D, LED_SMD:LED_SK6812_PLCC4_5.0x5.0mm_P3.2mm, symbol LED:SK6812
- added D5: SK6812_E, LED_SMD:LED_SK6812_PLCC4_5.0x5.0mm_P3.2mm, symbol LED:SK6812
- added D6: SK6812_F, LED_SMD:LED_SK6812_PLCC4_5.0x5.0mm_P3.2mm, symbol LED:SK6812
- added D7: SK6812_G, LED_SMD:LED_SK6812_PLCC4_5.0x5.0mm_P3.2mm, symbol LED:SK6812
- added D8: SK6812_H, LED_SMD:LED_SK6812_PLCC4_5.0x5.0mm_P3.2mm, symbol LED:SK6812
- added D9: SK6812_I, LED_SMD:LED_SK6812_PLCC4_5.0x5.0mm_P3.2mm, symbol LED:SK6812
- C1, C10, C11, C12, C13, C14, C15, C16, C2, C5, C6, C7, C8, C9: footprint (none) -> Capacitor_SMD:C_0805_2012Metric_Pad1.15x1.40mm_HandSolder
- C3: footprint (none) -> Capacitor_THT:CP_Radial_D10.0mm_P5.00mm_P7.50mm
- C4: footprint (none) -> Capacitor_THT:CP_Radial_D10.0mm_P2.50mm_P5.00mm
- J10, J8, J9: footprint (none) -> TerminalBlock:TerminalBlock_bornier-2_P5.08mm
- J4: value IOVCC -> 5V
- U10: value ULN2003AModule -> ULN2003A_E; footprint ULN2003AModule:ULN2003AModule -> ULN2003AModule:ULN2003AModule_No_EN; symbol ULN2003AModule:ULN2003AModule -> ULN2003AModule:ULN2003AModule_No_EN
- U12: value ULN2003AModule -> ULN2003A_D; footprint ULN2003AModule:ULN2003AModule -> ULN2003AModule:ULN2003AModule_No_EN; symbol ULN2003AModule:ULN2003AModule -> ULN2003AModule:ULN2003AModule_No_EN
- U13: value ULN2003AModule -> ULN2003A_C; footprint ULN2003AModule:ULN2003AModule -> ULN2003AModule:ULN2003AModule_No_EN; symbol ULN2003AModule:ULN2003AModule -> ULN2003AModule:ULN2003AModule_No_EN
- U14: value ULN2003AModule -> ULN2003A_B; footprint ULN2003AModule:ULN2003AModule -> ULN2003AModule:ULN2003AModule_No_EN; symbol ULN2003AModule:ULN2003AModule -> ULN2003AModule:ULN2003AModule_No_EN
- U15: value ULN2003AModule -> ULN2003A_A; footprint ULN2003AModule:ULN2003AModule -> ULN2003AModule:ULN2003AModule_No_EN; symbol ULN2003AModule:ULN2003AModule -> ULN2003AModule:ULN2003AModule_No_EN
- U2: footprint Connector_PinSocket_2.54mm:PinSocket_1x04_P2.54mm_Vertical -> SSD1306:SSD1306_128x32
- U3: value ULN2003AModule -> ULN2003A_L; footprint ULN2003AModule:ULN2003AModule -> ULN2003AModule:ULN2003AModule_No_EN; symbol ULN2003AModule:ULN2003AModule -> ULN2003AModule:ULN2003AModule_No_EN
- U4: value ULN2003AModule -> ULN2003A_K; footprint ULN2003AModule:ULN2003AModule -> ULN2003AModule:ULN2003AModule_No_EN; symbol ULN2003AModule:ULN2003AModule -> ULN2003AModule:ULN2003AModule_No_EN
- U5: value ULN2003AModule -> ULN2003A_J; footprint ULN2003AModule:ULN2003AModule -> ULN2003AModule:ULN2003AModule_No_EN; symbol ULN2003AModule:ULN2003AModule -> ULN2003AModule:ULN2003AModule_No_EN
- U6: value ULN2003AModule -> ULN2003A_I; footprint ULN2003AModule:ULN2003AModule -> ULN2003AModule:ULN2003AModule_No_EN; symbol ULN2003AModule:ULN2003AModule -> ULN2003AModule:ULN2003AModule_No_EN
- U7: value ULN2003AModule -> ULN2003A_H; footprint ULN2003AModule:ULN2003AModule -> ULN2003AModule:ULN2003AModule_No_EN; symbol ULN2003AModule:ULN2003AModule -> ULN2003AModule:ULN2003AModule_No_EN
- U8: value ULN2003AModule -> ULN2003A_G; footprint ULN2003AModule:ULN2003AModule -> ULN2003AModule:ULN2003AModule_No_EN; symbol ULN2003AModule:ULN2003AModule -> ULN2003AModule:ULN2003AModule_No_EN
- U9: value ULN2003AModule -> ULN2003A_F; footprint ULN2003AModule:ULN2003AModule -> ULN2003AModule:ULN2003AModule_No_EN; symbol ULN2003AModule:ULN2003AModule -> ULN2003AModule:ULN2003AModule_No_EN
Connections:
- net +12V: now also J10.2 (Pin_2); no longer J10.1 (Pin_1)
- net +12V_Monitored: now also J10.1 (Pin_1); no longer C16.2, J10.2 (Pin_2)
- net +5V: now also C10.2, C11.2, C12.2, C13.2, C14.2, C15.2, C16.2, C2.2, C5.2, C7.2, C8.2, C9.2, J4.1 (Pin_1), J4.10 (Pin_10), J4.11 (Pin_11), J4.12 (Pin_12), J4.2 (Pin_2), J4.3 (Pin_3), J4.4 (Pin_4), J4.5 (Pin_5), J4.6 (Pin_6), J4.7 (Pin_7), J4.8 (Pin_8), J4.9 (Pin_9), JP4.1 (A), JP5.1 (A), U11.VCC, U2.3 (VCC), U31.VCC, U33.5 (VS), D1.3 (VDD), D10.3 (VDD), D11.3 (VDD), D12.3 (VDD), D2.3 (VDD), D3.3 (VDD), D4.3 (VDD), D5.3 (VDD), D6.3 (VDD), D7.3 (VDD), D8.3 (VDD), D9.3 (VDD)
- net GND: now also C10.1, C11.1, C12.1, C13.1, C14.1, C15.1, C7.1, C8.1, C9.1, D1.1 (VSS), D10.1 (VSS), D11.1 (VSS), D12.1 (VSS), D2.1 (VSS), D3.1 (VSS), D4.1 (VSS), D5.1 (VSS), D6.1 (VSS), D7.1 (VSS), D8.1 (VSS), D9.1 (VSS); no longer C10.2, C11.2, C12.2, C13.2, C14.2, C15.2, C7.2, C8.2, C9.2
- net MOTOR_A_PHASE_A: now also U1.D13, U15.IN1; no longer U1.A0, U3.IN1
- net MOTOR_A_PHASE_B: now also U1.D12, U15.IN2; no longer U1.A1, U3.IN2
- net MOTOR_A_PHASE_C: now also U1.D11, U15.IN3; no longer U1.A2, U3.IN3
- net MOTOR_A_PHASE_D: now also U1.D10, U15.IN4; no longer U1.A3, U3.IN4
- net MOTOR_B_PHASE_A: now also U1.D25, U14.IN1; no longer U1.A4, U4.IN1
- net MOTOR_B_PHASE_B: now also U1.D24, U14.IN2; no longer U1.A5, U4.IN2
- net MOTOR_B_PHASE_C: now also U1.D23, U14.IN3; no longer U1.A6, U4.IN3
- net MOTOR_B_PHASE_D: now also U1.D22, U14.IN4; no longer U1.A7, U4.IN4
- net MOTOR_C_PHASE_A: now also U1.D29, U13.IN1; no longer U1.A8, U5.IN1
- net MOTOR_C_PHASE_B: now also U1.D28, U13.IN2; no longer U1.A9, U5.IN2
- net MOTOR_C_PHASE_C: now also U1.D27, U13.IN3; no longer U1.A10, U5.IN3
- net MOTOR_C_PHASE_D: now also U1.D26, U13.IN4; no longer U1.A11, U5.IN4
- net MOTOR_D_PHASE_A: now also U1.D30, U12.IN1; no longer U1.A12, U6.IN1
- net MOTOR_D_PHASE_B: now also U1.D31, U12.IN2; no longer U1.A13, U6.IN2
- net MOTOR_D_PHASE_C: now also U1.D32, U12.IN3; no longer U1.A14, U6.IN3
- net MOTOR_D_PHASE_D: now also U1.D33, U12.IN4; no longer U1.A15, U6.IN4
- net MOTOR_E_PHASE_A: now also U1.D34, U10.IN1; no longer U1.D53, U7.IN1
- net MOTOR_E_PHASE_B: now also U1.D35, U10.IN2; no longer U1.D52, U7.IN2
- net MOTOR_E_PHASE_C: now also U1.D36, U10.IN3; no longer U1.D51, U7.IN3
- net MOTOR_E_PHASE_D: now also U1.D37, U10.IN4; no longer U1.D50, U7.IN4
- net MOTOR_F_PHASE_A: now also U1.D42, U9.IN1; no longer U1.D49, U8.IN1
- net MOTOR_F_PHASE_B: now also U1.D43, U9.IN2; no longer U1.D48, U8.IN2
- net MOTOR_F_PHASE_C: now also U1.D44, U9.IN3; no longer U1.D47, U8.IN3
- net MOTOR_F_PHASE_D: now also U1.D45, U9.IN4; no longer U1.D46, U8.IN4
- net MOTOR_G_PHASE_A: now also U1.D46, U8.IN1; no longer U1.D45, U9.IN1
- net MOTOR_G_PHASE_B: now also U1.D47, U8.IN2; no longer U1.D44, U9.IN2
- net MOTOR_G_PHASE_C: now also U1.D48, U8.IN3; no longer U1.D43, U9.IN3
- net MOTOR_G_PHASE_D: now also U1.D49, U8.IN4; no longer U1.D42, U9.IN4
- net MOTOR_H_PHASE_A: now also U1.D50, U7.IN1; no longer U1.D37, U10.IN1
- net MOTOR_H_PHASE_B: now also U1.D51, U7.IN2; no longer U1.D36, U10.IN2
- net MOTOR_H_PHASE_C: now also U1.D52, U7.IN3; no longer U1.D35, U10.IN3
- net MOTOR_H_PHASE_D: now also U1.D53, U7.IN4; no longer U1.D34, U10.IN4
- net MOTOR_I_PHASE_A: now also U1.A15, U6.IN1; no longer U1.D33, U12.IN1
- net MOTOR_I_PHASE_B: now also U1.A14, U6.IN2; no longer U1.D32, U12.IN2
- net MOTOR_I_PHASE_C: now also U1.A13, U6.IN3; no longer U1.D31, U12.IN3
- net MOTOR_I_PHASE_D: now also U1.A12, U6.IN4; no longer U1.D30, U12.IN4
- net MOTOR_J_PHASE_A: now also U1.A11, U5.IN1; no longer U1.D29, U13.IN1
- net MOTOR_J_PHASE_B: now also U1.A10, U5.IN2; no longer U1.D28, U13.IN2
- net MOTOR_J_PHASE_C: now also U1.A9, U5.IN3; no longer U1.D27, U13.IN3
- net MOTOR_J_PHASE_D: now also U1.A8, U5.IN4; no longer U1.D26, U13.IN4
- net MOTOR_K_PHASE_A: now also U1.A7, U4.IN1; no longer U1.D25, U14.IN1
- net MOTOR_K_PHASE_B: now also U1.A6, U4.IN2; no longer U1.D24, U14.IN2
- net MOTOR_K_PHASE_C: now also U1.A5, U4.IN3; no longer U1.D23, U14.IN3
- net MOTOR_K_PHASE_D: now also U1.A4, U4.IN4; no longer U1.D22, U14.IN4
- net MOTOR_L_PHASE_A: now also U1.A3, U3.IN1; no longer U1.D10, U15.IN1
- net MOTOR_L_PHASE_B: now also U1.A2, U3.IN2; no longer U1.D11, U15.IN2
- net MOTOR_L_PHASE_C: now also U1.A1, U3.IN3; no longer U1.D12, U15.IN3
- net MOTOR_L_PHASE_D: now also U1.A0, U3.IN4; no longer U1.D13, U15.IN4
- net LED_SIGNAL: now reaches U1.D5
- net LED_SIGNAL: now also D1.2 (DIN)
- net RS485_B: now reaches J8.2 (Pin_2), J9.2 (Pin_2)
- net RS485_B: now also U32.7 (B); no longer U32.6 (A)
- net RS485_A: now reaches J8.1 (Pin_1), J9.1 (Pin_1)
- net RS485_A: now also U32.6 (A); no longer U32.7 (B)
- removed net IOVCC: C10.1, C11.1, C12.1, C13.1, C14.1, C15.1, C2.2, C5.2, C7.1, C8.1, C9.1, J4.1 (Pin_1), J4.10 (Pin_10), J4.11 (Pin_11), J4.12 (Pin_12), J4.2 (Pin_2), J4.3 (Pin_3), J4.4 (Pin_4), J4.5 (Pin_5), J4.6 (Pin_6), J4.7 (Pin_7), J4.8 (Pin_8), J4.9 (Pin_9), JP4.1 (A), JP5.1 (A), U1.IOREF, U11.VCC, U2.3 (VCC), U31.VCC, U33.5 (VS)
- new net: D1.4 (DOUT), D2.2 (DIN)
- new net: D2.4 (DOUT), D3.2 (DIN)
- new net: D3.4 (DOUT), D4.2 (DIN)
- new net: D4.4 (DOUT), D5.2 (DIN)
- new net: D5.4 (DOUT), D6.2 (DIN)
- new net: D6.4 (DOUT), D7.2 (DIN)
- new net: D7.4 (DOUT), D8.2 (DIN)
- new net: D8.4 (DOUT), D9.2 (DIN)
- new net: D10.2 (DIN), D9.4 (DOUT)
- new net: D10.4 (DOUT), D11.2 (DIN)
- new net: D11.4 (DOUT), D12.2 (DIN)
- no-connect marks 52 -> 22
Other:
- note added: "A"
- note added: "B"
- note added: "C"
- note added: "D"
- note added: "E"
- note added: "F"
- note added: "G"
- note added: "H"
- note added: "I"
- note added: "J"
- note added: "K"
- note added: "L"
- note removed: "47k. DNP for Mega 2560"
- note removed: "ESP32/ESP8266 IO Support"
- note removed: "For compatibility with ESP8266, all critical IO\nuses the inner pins; optional IO (e.g. display)\ncan use the outer pins (only present for ESP32\nmodules)"
- note removed: "IOVCC is sourced by the MCU\nmodule that's inserted, at the\nappropriate IO voltage\n(3.3V or 5V)"
- note removed: "MCU Option 2: TTGO T-Display (ESP32)"
- note removed: "MCU Option 3: ESP32/ESP8266 D1 Mini"
- note removed: "Optional: Shift register chaining support"

Commit message: Initial routing
Parts:
- C3: footprint Capacitor_THT:CP_Radial_D10.0mm_P5.00mm_P7.50mm -> Capacitor_THT:CP_Radial_D10.0mm_P3.50mm
- C4: footprint Capacitor_THT:CP_Radial_D10.0mm_P2.50mm_P5.00mm -> Capacitor_THT:CP_Radial_D6.3mm_P2.50mm
Connections:
- net SCL: now also U1.SCL (D21_SCL); no longer U1.D21
- net SDA: now also U1.SDA (D20_SDA); no longer U1.D20
- no-connect marks 22 -> 24
Other:
- note added: "Dedicated SDA/SCL pins are used,\nso these must be left disconnected."
- note removed: "A"
- note removed: "B"
- note removed: "C"
- note removed: "D"
- note removed: "E"
- note removed: "F"
- note removed: "G"
- note removed: "H"
- note removed: "I"
- note removed: "J"
- note removed: "K"
- note removed: "L"
Changed lines of the file:
@@
 NoConn ~ 19250 1800
 Wire Wire Line
-	19250 4900 19500 4900
-Wire Wire Line
-	19250 4800 19500 4800
-Text Label 19500 4800 2    50   ~ 0
+	19250 10100 19500 10100
+Wire Wire Line
+	19250 10000 19500 10000
+Text Label 19500 10000 2    50   ~ 0
 SDA
-Text Label 19500 4900 2    50   ~ 0
+Text Label 19500 10100 2    50   ~ 0
 SCL
 Wire Wire Line
@@
 F 0 "C3" H 4538 1296 50  0000 L CNN
 F 1 "100uF" H 4538 1205 50  0000 L CNN
-F 2 "Capacitor_THT:CP_Radial_D10.0mm_P5.00mm_P7.50mm" H 4450 1250 50  0001 C CNN
+F 2 "Capacitor_THT:CP_Radial_D10.0mm_P3.50mm" H 4450 1250 50  0001 C CNN
 F 3 "~" H 4450 1250 50  0001 C CNN
 	1    4450 1250
@@
 F 0 "C4" H 5088 1296 50  0000 L CNN
 F 1 "10uF" H 5088 1205 50  0000 L CNN
-F 2 "Capacitor_THT:CP_Radial_D10.0mm_P2.50mm_P5.00mm" H 5000 1250 50  0001 C CNN
+F 2 "Capacitor_THT:CP_Radial_D6.3mm_P2.50mm" H 5000 1250 50  0001 C CNN
 F 3 "~" H 5000 1250 50  0001 C CNN
 	1    5000 1250
@@
 Text Label 20100 8600 2    50   ~ 0
 MOTOR_L_PHASE_A
-Text Notes 20250 3950 0    50   ~ 0
-L
-Text Notes 20250 5100 0    50   ~ 0
-K
-Text Notes 20250 5500 0    50   ~ 0
-J
-Text Notes 20250 5850 0    50   ~ 0
-I
-Text Notes 20250 6350 0    50   ~ 0
-H
-Text Notes 20250 7150 0    50   ~ 0
-G
-Text Notes 20250 7550 0    50   ~ 0
-F
-Text Notes 20250 7900 0    50   ~ 0
-E
-Text Notes 20250 8450 0    50   ~ 0
-A
-Text Notes 20250 8850 0    50   ~ 0
-B
-Text Notes 20250 9250 0    50   ~ 0
-C
-Text Notes 20250 9650 0    50   ~ 0
-D
+NoConn ~ 19250 4800
+NoConn ~ 19250 4900
+Text Notes 19300 4900 0    50   ~ 0
+Dedicated SDA/SCL pins are used,\nso these must be left disconnected.
 $EndSCHEMATC
