File: electronics/espShifter/espShifter.kicad_pcb (KiCad board)
At the start: 2 copper layers, 100 x 100 mm, 89 parts, among them J1 Power In, J11 Motor A, J12 Motor E, J13 Motor I, J14 Motor B, J15 Motor F, J16 Motor J, J17 Motor C, J18 Motor G, J19 Motor K, J2 UART, J20 Motor D, J21 Motor H, J22 Motor L, J3 SENSOR, J4 IOVCC, J5 GND, J6 SR CHAIN IN, J7 SR CHAIN OUT, Q1 BSS138, Q2 BSS138, U1 Mega2560Shield, U10 ULN2003AModule, U11 INA219 Breakout Wide (blue), U12 ULN2003AModule, U13 ULN2003AModule, U14 ULN2003AModule, U15 ULN2003AModule, U16 LevelShifterModule, U17 RS485Module, U18 TTGO_TDisplay, U19 74HC244, U2 SSD1306_I2C, U20 74HC165, U21 74HC165, U22 ST7789_80x160, U23 D1_32, U24 74HC595, U25 74HC595, U26 74HC595, U27 74HC595, U28 74HC595, U29 74HC595, U3 ULN2003AModule, U30 ST7789_240x240, U31 INA219 Breakout Narrow (purpl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, U32 SP485, U33 INA219BxD, U34 TPL7407LA, U35 TPL7407LA, U36 TPL7407LA, U37 TPL7407LA, U38 TPL7407LA, U39 TPL7407LA, U4 ULN2003AModule, U40 TPL7407LA, U5 ULN2003AModule, U6 ULN2003AModule, U7 ULN2003AModule, U8 ULN2003AModule, U9 ULN2003AModule

Commit message: WIP ESP PCB
Parts:
- removed JP1: 12V_VIN, Connector_PinHeader_2.54mm:PinHeader_1x02_P2.54mm_Vertical
- removed R10, R11, R12, R2, R3, R4, R5, R6, R7, R8, R9: 47k, Resistor_THT:R_Axial_DIN0204_L3.6mm_D1.6mm_P1.90mm_Vertical
- removed U1: Mega2560Shield, Mega2560Shield:Mega2560Shield
- removed U10, U12, U13, U14, U15, U3, U4, U5, U6, U7, U8, U9: ULN2003AModule, ULN2003AModule:ULN2003AModule
- removed U17: RS485Module, RS485:RS485Module
- added C1: 0.1uF, Capacitor_SMD:C_0805_2012Metric, F.Cu at (76.7, -22.9)
- added C10: 0.1uF, Capacitor_SMD:C_0805_2012Metric, F.Cu at (69.9, -18.8)
- added C11: 0.1uF, Capacitor_SMD:C_0805_2012Metric, F.Cu at (60.6, -8.51)
- added C12: 0.1uF, Capacitor_SMD:C_0805_2012Metric, F.Cu at (66.1, -9.06)
- added C13: 0.1uF, Capacitor_SMD:C_0805_2012Metric, F.Cu at (74.3, -18.8)
- added C14: 0.1uF, Capacitor_SMD:C_0805_2012Metric, F.Cu at (69.9, -15.9)
- added C15: 0.1uF, Capacitor_SMD:C_0805_2012Metric, F.Cu at (43.0, -8.51)
- added C16: 0.1uF, Capacitor_SMD:C_0805_2012Metric, F.Cu at (74.3, -15.9)
- added C17: 0.1uF, Capacitor_SMD:C_0805_2012Metric, F.Cu at (69.9, -12.9)
- added C18: 0.1uF, Capacitor_SMD:C_0805_2012Metric, F.Cu at (78.7, -19.9)
- added C19: 0.1uF, Capacitor_SMD:C_0805_2012Metric, F.Cu at (70.5, -9.96)
- added C2: 0.1uF, Capacitor_SMD:C_0805_2012Metric, F.Cu at (47.4, -8.51)
- added C20: 0.1uF, Capacitor_SMD:C_0805_2012Metric, F.Cu at (74.3, -12.9)
- added C21: 0.1uF, Capacitor_SMD:C_0805_2012Metric, F.Cu at (78.7, -17.0)
- added C22: 0.1uF, Capacitor_SMD:C_0805_2012Metric, F.Cu at (70.5, -7.01)
- added C3: 100uF, Capacitor_SMD:CP_Elec_8x10.5, F.Cu at (47.5, -24.1)
- added C4: 10uF, Capacitor_SMD:CP_Elec_4x5.4, F.Cu at (69.6, -26.2)
- added C5: 0.1uF, Capacitor_SMD:C_0805_2012Metric, F.Cu at (67.9, -21.8)
- added C6: 0.1uF, Capacitor_SMD:C_0805_2012Metric, F.Cu at (51.8, -8.51)
- added C7: 0.1uF, Capacitor_SMD:C_0805_2012Metric, F.Cu at (79.5, -27.6)
- added C8: 0.1uF, Capacitor_SMD:C_0805_2012Metric, F.Cu at (56.2, -8.51)
- added C9: 0.1uF, Capacitor_SMD:C_0805_2012Metric, F.Cu at (72.3, -21.8)
- added J10: 12V SENSE, TerminalBlock:TerminalBlock_bornier-2_P5.08mm, F.Cu at (55.6, -14.5)
- added J8: RS485, TerminalBlock:TerminalBlock_bornier-2_P5.08mm, F.Cu at (44.0, -14.5)
- added J9: RS485, TerminalBlock:TerminalBlock_bornier-2_P5.08mm, F.Cu at (57.4, -24.6)
- added RN1: 47k, Resistor_SMD:R_Cat16-4, F.Cu at (75.3, -26.7)
- added RN2: 47k, Resistor_SMD:R_Cat16-4, F.Cu at (65.8, -12.9)
- added RN3: 47k, Resistor_SMD:R_Cat16-4, F.Cu at (65.8, -17.7)
- H1, H2, H3, H4: footprint MountingHole:MountingHole_4.3mm_M4_ISO7380 -> MountingHole:MountingHole_4.3mm_M4_ISO7380_Pad
- J1: footprint TerminalBlock:TerminalBlock_bornier-3_P5.08mm -> TerminalBlock:TerminalBlock_bornier-4_P5.08mm
- J4: value IOVCC -> 3.3v
- JP2: value RX 3.3V -> RX BYPASS
- JP3: value TX 3.3V -> TX BYPASS
- R1: value 47k -> 10k; footprint Resistor_THT:R_Axial_DIN0204_L3.6mm_D1.6mm_P1.90mm_Vertical -> Resistor_SMD:R_0805_2012Metric
- R13, R14, R15, R16, R17, R18: footprint Resistor_SMD:R_0805_2012Metric_Pad1.15x1.40mm_HandSolder -> Resistor_SMD:R_0805_2012Metric
- U19: footprint Package_DIP:DIP-20_W7.62mm -> Package_SO:TSSOP-20_4.4x6.5mm_P0.65mm
- U20, U21, U24, U25, U26, U27, U28, U29: footprint Package_DIP:DIP-16_W7.62mm -> Package_SO:SOIC-16_3.9x9.9mm_P1.27mm
- moved R1 208.1 mm to (74.9, -9.96)
- moved U18 91.8 mm to (-25.4, 5.59), turned to 0 degrees
- moved U23 66.3 mm to (8.38, 31.5), turned to 180 degrees
Connections:
- J4 pad 1: IOVCC -> +3V3
- J4 pad 10: IOVCC -> +3V3
- J4 pad 11: IOVCC -> +3V3
- J4 pad 12: IOVCC -> +3V3
- J4 pad 2: IOVCC -> +3V3
- J4 pad 3: IOVCC -> +3V3
- J4 pad 4: IOVCC -> +3V3
- J4 pad 5: IOVCC -> +3V3
- J4 pad 6: IOVCC -> +3V3
- J4 pad 7: IOVCC -> +3V3
- J4 pad 8: IOVCC -> +3V3
- J4 pad 9: IOVCC -> +3V3
- JP4 pad 1: IOVCC -> +3V3
- JP5 pad 1: IOVCC -> +3V3
- Q1 pad 1: IOVCC -> +3V3
- Q2 pad 1: IOVCC -> +3V3
- R1 pad 1: IOVCC -> /SENSOR_DATA_CHAIN
- R1 pad 2: /SENSOR_A -> GND
- R13 pad 1: IOVCC -> +3V3
- R14 pad 1: IOVCC -> +3V3
- U11 pad GND: (no net) -> GND
- U11 pad SCL: (no net) -> /SCL
- U11 pad SDA: (no net) -> /SDA
- U11 pad VCC: (no net) -> +3V3
- U16 pad 3: IOVCC -> +3V3
- U18 pad 12: IOVCC -> +3V3
- U18 pad 24: IOVCC -> +3V3
- U19 pad 20: IOVCC -> +3V3
- U2 pad 3: IOVCC -> +3V3
- U20 pad 16: IOVCC -> +3V3
- U21 pad 16: IOVCC -> +3V3
- U22 pad VCC: IOVCC -> +3V3
- U23 pad 16: IOVCC -> +3V3
- U24 pad 10: IOVCC -> +3V3
- U24 pad 16: IOVCC -> +3V3
- U25 pad 10: IOVCC -> +3V3
- U25 pad 16: IOVCC -> +3V3
- U26 pad 10: IOVCC -> +3V3
- U26 pad 16: IOVCC -> +3V3
- U27 pad 10: IOVCC -> +3V3
- U27 pad 16: IOVCC -> +3V3
- U28 pad 10: IOVCC -> +3V3
- U28 pad 16: IOVCC -> +3V3
- U29 pad 10: IOVCC -> +3V3
- U29 pad 16: IOVCC -> +3V3
- U30 pad VCC: IOVCC -> +3V3
- U31 pad GND: (no net) -> GND
- U31 pad SCL: (no net) -> /SCL
- U31 pad SDA: (no net) -> /SDA
- U31 pad VCC: (no net) -> +3V3
- U32 pad 6: (no net) -> Net-(J8-Pad2)
- U32 pad 7: (no net) -> Net-(J8-Pad1)
- U33 pad 5: IOVCC -> +3V3

Commit message: WIP PCB Layout
Parts:
- removed the J13 at (354.8, 119.5)
- removed the J16 at (405.0, 74.3)
- added J18: Motor H, JST_XH_Connectors:JST_XH_2-5mm_5pin, F.Cu at (43.2, 50.8)
- added J20: Motor J, JST_XH_Connectors:JST_XH_2-5mm_5pin, F.Cu at (73.7, 50.8)
- J19: value Motor K -> Motor I
- J21: value Motor H -> Motor K
- moved J11 381.6 mm to (27.9, 22.9)
- moved U24 374.7 mm to (48.3, 38.1), turned to 90 degrees
- moved U37 352.7 mm to (73.7, 58.4), turned to 90 degrees
- moved U34 350.6 mm to (35.6, 30.5), turned to 90 degrees
- moved U38 343.6 mm to (83.8, 30.5), turned to 90 degrees
- moved J14 342.4 mm to (73.7, 22.9)
- moved J12 328.3 mm to (43.2, 22.9)
- moved U35 323.7 mm to (50.8, 58.4), turned to 90 degrees
- moved U36 319.1 mm to (59.7, 30.5), turned to 90 degrees
- moved J16 313.0 mm to (104.1, 22.9)
- moved J13 307.6 mm to (58.4, 22.9)
- moved J19 300.6 mm to (58.4, 50.8)
- moved J21 294.0 mm to (88.9, 50.8)
- moved J15 280.6 mm to (88.9, 22.9)
- moved J17 269.4 mm to (119.4, 22.9)
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- renumbered J14 to J12, J17 to J13, J20 to J14, J12 to J15, J15 to J16, J18 to J17
Connections:
- J19 pad 1: /OUT_K_PHASE_A -> /OUT_I_PHASE_A
- J19 pad 2: /OUT_K_PHASE_B -> /OUT_I_PHASE_B
- J19 pad 3: /OUT_K_PHASE_C -> /OUT_I_PHASE_C
- J19 pad 4: /OUT_K_PHASE_D -> /OUT_I_PHASE_D
- J21 pad 1: /OUT_H_PHASE_A -> /OUT_K_PHASE_A
- J21 pad 2: /OUT_H_PHASE_B -> /OUT_K_PHASE_B
- J21 pad 3: /OUT_H_PHASE_C -> /OUT_K_PHASE_C
- J21 pad 4: /OUT_H_PHASE_D -> /OUT_K_PHASE_D
Other:
- board size 100 x 100 mm -> 100 x 105.1 mm
