File: electronics/chainlinkBase/chainlinkBase.kicad_pcb (KiCad board)
At the start: 2 copper layers, 100 x 105.1 mm, 91 parts, among them J1 Power In, J10 12V SENSE, J11 Motor A, J12 Motor B, J13 Motor C, J14 Motor D, J15 Motor E, J16 Motor F, J17 Motor G, J18 Motor H, J19 Motor I, J2 UART, J20 Motor J, J21 Motor K, J22 Motor L, J3 SENSOR, J4 3.3v, J5 GND, J6 SR CHAIN IN, J7 SR CHAIN OUT, J8 RS485, J9 RS485, Q1 BSS138, Q2 BSS138, U11 INA219 Breakout Wide (blue), U16 LevelShifterModule, U18 TTGO_TDisplay, U19 74HC244, U2 SSD1306_I2C, U20 74HC165, U21 74HC165, U22 ST7789_80x160, U23 D1_32, U24 74HC595, U25 74HC595, U26 74HC595, U27 74HC595, U28 74HC595, U29 74HC595, U30 ST7789_240x240, U31 INA219 Breakout Narrow (purpl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, U32 SP485, U33 INA219BxD, U34 TPL7407LA, U35 TPL7407LA, U36 TPL7407LA, U37 TPL7407LA, U38 TPL7407LA, U39 TPL7407LA, U40 TPL7407LA

Commit message: checkpoint - more component selection and schematic work
Parts:
- removed the C22 at (70.5, -7.01)
- removed C4: 10uF, Capacitor_SMD:CP_Elec_4x5.4
- removed the C5 at (67.9, -21.8)
- removed H1, H2, H3, H4: MountingHole, MountingHole:MountingHole_4.3mm_M4_ISO7380_Pad
- removed J14: Motor D, JST_XH_Connectors:JST_XH_2-5mm_5pin
- removed J15: Motor E, JST_XH_Connectors:JST_XH_2-5mm_5pin
- removed J16: Motor F, JST_XH_Connectors:JST_XH_2-5mm_5pin
- removed J17: Motor G, JST_XH_Connectors:JST_XH_2-5mm_5pin
- removed J18: Motor H, JST_XH_Connectors:JST_XH_2-5mm_5pin
- removed J19: Motor I, JST_XH_Connectors:JST_XH_2-5mm_5pin
- removed J20: Motor J, JST_XH_Connectors:JST_XH_2-5mm_5pin
- removed J21: Motor K, JST_XH_Connectors:JST_XH_2-5mm_5pin
- removed J22: Motor L, JST_XH_Connectors:JST_XH_2-5mm_5pin
- removed the J6 at (178.3, -7.09)
- removed the J7 at (182.9, -7.09)
- removed JP2: RX BYPASS, Jumper:SolderJumper-2_P1.3mm_Open_TrianglePad1.0x1.5mm
- removed JP3: TX BYPASS, Jumper:SolderJumper-2_P1.3mm_Open_TrianglePad1.0x1.5mm
- removed JP4: A0, Jumper:SolderJumper-2_P1.3mm_Open_TrianglePad1.0x1.5mm
- removed JP5: A1, Jumper:SolderJumper-2_P1.3mm_Open_TrianglePad1.0x1.5mm
- removed Q1, Q2: BSS138, Package_TO_SOT_SMD:SOT-23
- removed R19: 0.1R 1% 1/2 W, Resistor_SMD:R_2512_6332Metric_Pad1.52x3.35mm_HandSolder
- removed RN1, RN2, RN3: 47k, Resistor_SMD:R_Cat16-4
- removed U19: 74HC244, Package_SO:TSSOP-20_4.4x6.5mm_P0.65mm
- removed U20, U21: 74HC165, Package_SO:SOIC-16_3.9x9.9mm_P1.27mm
- removed U22: ST7789_80x160, ST7789:ST7789_80x160
- removed U23: D1_32, ESP32:D1_32
- removed U24, U25, U26, U27, U28, U29: 74HC595, Package_SO:SOIC-16_3.9x9.9mm_P1.27mm
- removed U30: ST7789_240x240, ST7789:ST7789_240x240
- removed U31: INA219 Breakout Narrow (purple), INA219:INA219_SMALL
- removed U34, U35, U36, U37, U38, U39, U40: TPL7407LA, Package_SO:SOIC-16_3.9x9.9mm_P1.27mm
- added C2: 4.7uF, Capacitor_SMD:C_0805_2012Metric, F.Cu at (113.7, -70.5)
- added C23: 0.1uF, Capacitor_SMD:C_0805_2012Metric, F.Cu at (87.5, -38.3)
- added C24: 0.1uF, Capacitor_SMD:C_0805_2012Metric, F.Cu at (95.1, -47.9)
- added C25: 1uF, Capacitor_SMD:C_0805_2012Metric, F.Cu at (99.5, -47.9)
- added C26: 1uF, Capacitor_SMD:C_0805_2012Metric, F.Cu at (95.1, -50.9)
- added C27: 0.1uF, Capacitor_SMD:C_0805_2012Metric, F.Cu at (101.2, -55.6)
- added C28: 0.1uF, Capacitor_SMD:C_0805_2012Metric, F.Cu at (113.7, -67.5)
- added C29: 0.1uF, Capacitor_SMD:C_0805_2012Metric, F.Cu at (87.9, -42.0)
- added C30: 0.1uF, Capacitor_SMD:C_0805_2012Metric, F.Cu at (109.8, -64.4)
- added C31: 0.1uF, Capacitor_SMD:C_0805_2012Metric, F.Cu at (83.0, -38.3)
- added C32: 0.1uF, Capacitor_SMD:C_0805_2012Metric, F.Cu at (87.9, -45.0)
- added C33: 0.1uF, Capacitor_SMD:C_0805_2012Metric, F.Cu at (90.6, -48.0)
- added D1: LED_Small, LED_SMD:LED_0805_2012Metric, F.Cu at (116.0, -75.1)
- added D10: WS2812B, LED_SMD:LED_WS2812B_PLCC4_5.0x5.0mm_P3.2mm, F.Cu at (104.2, -76.3)
- added D11: WS2812B, LED_SMD:LED_WS2812B_PLCC4_5.0x5.0mm_P3.2mm, F.Cu at (72.2, -41.1)
- added D2: LED_Small, LED_SMD:LED_0805_2012Metric, F.Cu at (101.2, -58.6)
- added D3: LED_Small, LED_SMD:LED_0805_2012Metric, F.Cu at (83.5, -41.4)
- added D4: LED_Small, LED_SMD:LED_0805_2012Metric, F.Cu at (96.4, -54.0)
- added D5: LED_Small, LED_SMD:LED_0805_2012Metric, F.Cu at (109.2, -67.5)
- added D6: WS2812B, LED_SMD:LED_WS2812B_PLCC4_5.0x5.0mm_P3.2mm, F.Cu at (78.8, -49.2)
- added D7: WS2812B, LED_SMD:LED_WS2812B_PLCC4_5.0x5.0mm_P3.2mm, F.Cu at (89.9, -55.8)
- added D8: WS2812B, LED_SMD:LED_WS2812B_PLCC4_5.0x5.0mm_P3.2mm, F.Cu at (102.8, -68.1)
- added D9: WS2812B, LED_SMD:LED_WS2812B_PLCC4_5.0x5.0mm_P3.2mm, F.Cu at (94.4, -68.1)
- added J2: CHANNEL, TerminalBlock:TerminalBlock_bornier-2_P5.08mm, F.Cu at (176.5, 57.1)
- added J8: Logic Power Out, TerminalBlock:TerminalBlock_bornier-2_P5.08mm, F.Cu at (70.3, -66.1)
- added R10: 0.01R 1% 1W, Resistor_SMD:R_0612_1632Metric, F.Cu at (174.2, 35.6)
- added R11: 0.01R 1% 1W, Resistor_SMD:R_0612_1632Metric, F.Cu at (178.3, 35.6)
- added R12: 10k, Resistor_SMD:R_0805_2012Metric, F.Cu at (110.1, -58.4)
- added R2: 0.01R 1% 1W, Resistor_SMD:R_0612_1632Metric, F.Cu at (170.2, 35.6)
- added R3: 2.2k, Resistor_SMD:R_0805_2012Metric, F.Cu at (110.1, -55.5)
- added R4: 2.2k, Resistor_SMD:R_0805_2012Metric, F.Cu at (96.8, -42.0)
- added R5: 10k, Resistor_SMD:R_0805_2012Metric, F.Cu at (118.7, -66.1)
- added R6: 10k, Resistor_SMD:R_0805_2012Metric, F.Cu at (104.0, -51.3)
- added R7: 220, Resistor_SMD:R_0805_2012Metric, F.Cu at (114.5, -61.5)
- added R8: 220, Resistor_SMD:R_0805_2012Metric, F.Cu at (91.9, -38.9)
- added R9: 10k, Resistor_SMD:R_0805_2012Metric, F.Cu at (96.8, -44.9)
- added SW1: SW_DIP_x04, Button_Switch_SMD:SW_DIP_SPSTx04_Slide_Omron_A6H-4101_W6.15mm_P1.27mm, F.Cu at (115.6, 78.7)
- added U1: AP7361C-33E, Package_TO_SOT_SMD:SOT-223-3_TabPin2, F.Cu at (64.8, 34.3)
- added U10: INA219BxD, Package_SO:SOIC-8_3.9x4.9mm_P1.27mm, F.Cu at (143.5, 118.1)
- added U12: NCP45560-H, Package_DFN_QFN:DFN-12-1EP_3x3mm_P0.5mm_EP2.05x2.86mm, F.Cu at (162.6, 115.6)
- added U13: SN74LV1T34DBV, Package_TO_SOT_SMD:SOT-23-5, F.Cu at (78.8, -43.6)
- added U15: INA219BxD, Package_SO:SOIC-8_3.9x4.9mm_P1.27mm, F.Cu at (143.5, 132.1)
- added U17: SN74LV1T34DBV, Package_TO_SOT_SMD:SOT-23-5, F.Cu at (96.5, -57.8)
- added U4: INA219BxD, Package_SO:SOIC-8_3.9x4.9mm_P1.27mm, F.Cu at (143.5, 64.8)
- added U5: NCP45560-H, Package_DFN_QFN:DFN-12-1EP_3x3mm_P0.5mm_EP2.05x2.86mm, F.Cu at (162.6, 50.8)
- added U6: NCP45560-H, Package_DFN_QFN:DFN-12-1EP_3x3mm_P0.5mm_EP2.05x2.86mm, F.Cu at (161.3, 69.8)
- added U8: MCP23017_SO, Package_SO:SSOP-28_5.3x10.2mm_P0.65mm, F.Cu at (101.6, 85.1)
- added U9: INA219BxD, Package_SO:SOIC-8_3.9x4.9mm_P1.27mm, F.Cu at (143.5, 105.4)
- C10, C11, C12, C17, C18, C19, C20, C9: value 0.1uF -> 1uF
- C3: value 100uF -> 4.7uF; footprint Capacitor_SMD:CP_Elec_8x10.5 -> Capacitor_SMD:C_0805_2012Metric
- J1: footprint TerminalBlock:TerminalBlock_bornier-4_P5.08mm -> TerminalBlock:TerminalBlock_bornier-2_P5.08mm
- J10: value 12V SENSE -> Output
- J11: value Motor A -> Output; footprint JST_XH_Connectors:JST_XH_2-5mm_5pin -> TerminalBlock:TerminalBlock_bornier-2_P5.08mm
- J12: value Motor B -> Output; footprint JST_XH_Connectors:JST_XH_2-5mm_5pin -> TerminalBlock:TerminalBlock_bornier-2_P5.08mm
- J13: value Motor C -> CHANNEL; footprint JST_XH_Connectors:JST_XH_2-5mm_5pin -> TerminalBlock:TerminalBlock_bornier-2_P5.08mm
- J3: value SENSOR -> CHANNEL; footprint Connector_PinHeader_2.54mm:PinHeader_1x12_P2.54mm_Vertical -> TerminalBlock:TerminalBlock_bornier-2_P5.08mm
- J4: value 3.3v -> CHANNEL; footprint Connector_PinHeader_2.54mm:PinHeader_1x12_P2.54mm_Vertical -> TerminalBlock:TerminalBlock_bornier-2_P5.08mm
- J5: value GND -> CHANNEL; footprint Connector_PinHeader_2.54mm:PinHeader_1x12_P2.54mm_Vertical -> TerminalBlock:TerminalBlock_bornier-2_P5.08mm
- R1, R16: value 10k -> 0.01R 1% 1W; footprint Resistor_SMD:R_0805_2012Metric -> Resistor_SMD:R_0612_1632Metric
- R14, R15, R18: value 10k -> 220
- U11: value INA219 Breakout Wide (blue) -> NCP45560-H; footprint INA219:INA219_LARGE -> Package_DFN_QFN:DFN-12-1EP_3x3mm_P0.5mm_EP2.05x2.86mm
- U16: value LevelShifterModule -> NCP45560-H; footprint LevelShifterModule:LevelShifterModule -> Package_DFN_QFN:DFN-12-1EP_3x3mm_P0.5mm_EP2.05x2.86mm
- U2: value SSD1306_I2C -> TPL7407LA; footprint Connector_PinSocket_2.54mm:PinSocket_1x04_P2.54mm_Vertical -> ModifiedSymbols:SOIC-16_3.9x9.9mm_P1.27mm_silk
- moved R17 261.2 mm to (101.2, -44.9)
- moved R18 255.4 mm to (114.5, -58.5)
- moved R14 254.4 mm to (104.0, -48.3)
- moved R15 253.6 mm to (96.3, -38.9)
- moved U2 244.3 mm to (82.8, -64.9)
- moved U14 197.8 mm to (73.7, 151.1), turned to 180 degrees
- moved J1 189.8 mm to (49.5, 26.7), turned to 180 degrees
- moved J7 178.9 mm to (56.5, 154.3), turned to 270 degrees
- moved R13 159.3 mm to (78.6, -36.7)
- moved J6 159.1 mm to (56.5, 144.1), turned to 270 degrees
- moved R16 147.1 mm to (182.3, 35.6)
- moved J13 144.1 mm to (176.5, 105.4), turned to 90 degrees
- moved J9 121.7 mm to (169.1, -69.3)
- moved R1 108.9 mm to (162.6, 54.6), turned to 90 degrees
- moved U16 99.2 mm to (165.1, 102.9)
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- renumbered C1 to C22, C2 to C5, J8 to J6, J9 to J7, J2 to J9, U32 to U14, U33 to U3, U18 to U7
Connections:
- C10 pad 1: +3V3 -> Net-(C10-Pad1)
- C11 pad 1: +3V3 -> Net-(C11-Pad1)
- C12 pad 1: +3V3 -> Net-(C12-Pad1)
- C13 pad 1: +3V3 -> GND
- C13 pad 2: GND -> +3V3
- C14 pad 1: +3V3 -> GND
- C14 pad 2: GND -> +3V3
- C16 pad 1: GND -> +3V3
- C16 pad 2: +12V_Monitored -> GND
- C17 pad 1: GND -> Net-(C17-Pad1)
- C17 pad 2: +12V_Monitored -> GND
- C18 pad 1: GND -> Net-(C18-Pad1)
- C18 pad 2: +12V_Monitored -> GND
- C19 pad 1: GND -> Net-(C19-Pad1)
- C19 pad 2: +12V_Monitored -> GND
- C20 pad 1: GND -> Net-(C20-Pad1)
- C20 pad 2: +12V_Monitored -> GND
- C21 pad 1: GND -> +3V3
- C21 pad 2: +12V_Monitored -> GND
- C3 pad 1: +12V -> /3V3_EXT
- C6 pad 2: +5V -> +3V3
- C9 pad 1: +3V3 -> Net-(C9-Pad1)
- J1 pad 1: +12V -> +5V
- J10 pad 1: +12V -> /CLOCK
- J10 pad 2: +12V_Monitored -> /MOTOR_DATA
- J11 pad 1: /OUT_A_PHASE_A -> /SENSOR_DATA
- J11 pad 2: /OUT_A_PHASE_B -> /LATCH
- J12 pad 1: /OUT_B_PHASE_A -> (no net)
- J12 pad 2: /OUT_B_PHASE_B -> GND
- J13 pad 1: /OUT_C_PHASE_A -> (no net)
- J13 pad 2: /OUT_C_PHASE_B -> Net-(C26-Pad1)
- J3 pad 1: /SENSOR_A -> (no net)
- J3 pad 2: /SENSOR_B -> Net-(C12-Pad1)
- J4 pad 1: +3V3 -> (no net)
- J4 pad 2: +3V3 -> Net-(C18-Pad1)
- J5 pad 1: GND -> (no net)
- J5 pad 2: GND -> Net-(C20-Pad1)
- J9 pad 1: /TX_EXT -> /TX
- J9 pad 2: /RX_EXT -> /RX
- R1 pad 1: /SENSOR_DATA_CHAIN -> Net-(F1-Pad1)
- R1 pad 2: GND -> Net-(C9-Pad1)
- R13 pad 1: +3V3 -> GND
- R13 pad 2: /RX -> /OUT3_EN
- R14 pad 1: +3V3 -> GND
- R14 pad 2: /TX -> Net-(D3-Pad1)
- R15 pad 1: +5V -> GND
- R15 pad 2: /RX_EXT -> Net-(D4-Pad1)
- R16 pad 1: +5V -> Net-(F5-Pad1)
- R16 pad 2: /TX_EXT -> Net-(C25-Pad1)
- R17 pad 1: Net-(JP4-Pad2) -> GND
- R17 pad 2: GND -> /OUT4_EN
- R18 pad 1: Net-(JP5-Pad2) -> GND
- R18 pad 2: GND -> Net-(D5-Pad1)
- U14 pad 1: /RX_EXT -> Net-(U13-Pad2)
- U14 pad 4: /TX_EXT -> /TX
- U16 pad 1: /RX -> Net-(C25-Pad1)
- U16 pad 10: +5V -> Net-(C26-Pad1)
- U16 pad 11: /TX_EXT -> Net-(C26-Pad1)
- U16 pad 12: /RX_EXT -> Net-(C26-Pad1)
- U16 pad 2: /TX -> /OUT4_EN
- U16 pad 6: (no net) -> /OUT4_PG
- U16 pad 7: (no net) -> Net-(C26-Pad1)
- U16 pad 8: (no net) -> Net-(C26-Pad1)
- U16 pad 9: GND -> Net-(C26-Pad1)
- U2 pad 1: /SDA -> /MASTER_EN
- U2 pad 2: /SCL -> /OUT0_EN
- U2 pad 3: +3V3 -> /OUT1_EN
- U2 pad 4: GND -> /OUT2_EN
- U3 pad 1: Net-(JP5-Pad2) -> GND
- U3 pad 2: Net-(JP4-Pad2) -> GND
- U3 pad 7: +12V_Monitored -> Net-(C9-Pad1)
- U3 pad 8: +12V -> Net-(F1-Pad1)
- U7 pad 15: /MOTOR_OE -> /RGB_LEDS_3V3
- U7 pad 16: /SENSOR_LATCH -> /MCP_RESET
- U7 pad 17: /MOTOR_LATCH -> /LATCH
- U7 pad 22: (no net) -> /MCP_INT
- U7 pad 23: (no net) -> /RX
- U7 pad 3: /RX -> /MASTER_EN
Other:
- board outline removed

Commit message: Switch to VN7007ALHTR for load switches
Parts:
- removed the C13 at (105.6, -54.2)
- removed the C14 at (105.3, -63.3)
- removed the C17 at (92.3, -44.9)
- removed the C18 at (114.2, -64.5)
- removed the C19 at (99.5, -50.9)
- removed the C20 at (105.6, -57.3)
- removed the C23 at (87.5, -38.3)
- removed C24: 0.1uF, Capacitor_SMD:C_0805_2012Metric
- removed C25, C26: 1uF, Capacitor_SMD:C_0805_2012Metric
- removed the J13 at (176.5, 105.4)
- removed the R13 at (78.6, -36.7)
- removed the R6 at (104.0, -51.3)
- added J14: CHANNEL, TerminalBlock:TerminalBlock_bornier-2_P5.08mm, F.Cu at (166.4, -4.70)
- added J6: CHANNEL, TerminalBlock:TerminalBlock_bornier-2_P5.08mm, F.Cu at (153.2, 12.5)
- added R19: 15k, Resistor_SMD:R_0805_2012Metric, F.Cu at (181.3, 16.7)
- added R20: 220, Resistor_SMD:R_0805_2012Metric, F.Cu at (192.7, 7.70)
- added R21: 220, Resistor_SMD:R_0805_2012Metric, F.Cu at (188.6, 13.7)
- added R22: 1k, Resistor_SMD:R_0805_2012Metric, F.Cu at (181.3, 19.7)
- added R23: 1k, Resistor_SMD:R_0805_2012Metric, F.Cu at (192.6, 10.7)
- added R24: 0.01R 1% 1W, Resistor_SMD:R_0612_1632Metric, F.Cu at (163.8, 20.4)
- added R25: 15k, Resistor_SMD:R_0805_2012Metric, F.Cu at (185.8, 16.7)
- added R26: 15k, Resistor_SMD:R_0805_2012Metric, F.Cu at (183.8, 10.8)
- added R27: 220, Resistor_SMD:R_0805_2012Metric, F.Cu at (181.3, 22.6)
- added R28: 1k, Resistor_SMD:R_0805_2012Metric, F.Cu at (188.2, 10.8)
- added R4: 15k, Resistor_SMD:R_0805_2012Metric, F.Cu at (172.5, 22.4)
- added R7: 15k, Resistor_SMD:R_0805_2012Metric, F.Cu at (176.9, 18.3)
- C10, C11, C12, C9: value 1uF -> 0.1uF
- J4: value CHANNEL -> RELAY
- R10: value 0.01R 1% 1W -> 220; footprint Resistor_SMD:R_0612_1632Metric -> Resistor_SMD:R_0805_2012Metric
- R11: value 0.01R 1% 1W -> 1k; footprint Resistor_SMD:R_0612_1632Metric -> Resistor_SMD:R_0805_2012Metric
- R12: value 10k -> 1k
- R14, R15: value 220 -> 0.01R 1% 1W; footprint Resistor_SMD:R_0805_2012Metric -> Resistor_SMD:R_0612_1632Metric
- R16: value 0.01R 1% 1W -> 15k; footprint Resistor_SMD:R_0612_1632Metric -> Resistor_SMD:R_0805_2012Metric
- R17: value 10k -> 15k
- R18, R8: value 220 -> 15k
- R3: renamed from R5; value 10k -> 15k
- R5: renamed from R3; value 2.2k -> 1k
- R6: renamed from R4; value 2.2k -> 1k
- SW1: footprint Button_Switch_SMD:SW_DIP_SPSTx04_Slide_Omron_A6H-4101_W6.15mm_P1.27mm -> Button_Switch_SMD:SW_DIP_SPSTx04_Slide_Omron_A6S-410x_W8.9mm_P2.54mm
- U11, U12, U16, U5, U6: value NCP45560-H -> VN7007ALH; footprint Package_DFN_QFN:DFN-12-1EP_3x3mm_P0.5mm_EP2.05x2.86mm -> VN7007ALHTR:VN7007ALHTR
- U8: value MCP23017_SO -> MCP23017_SS
- moved C6 121.9 mm to (194.3, -1.27)
- moved J5 116.7 mm to (166.4, 4.35), turned to 0 degrees
- moved U12 113.4 mm to (144.4, 3.67)
- moved U15 112.3 mm to (141.0, 19.8)
- moved D3 110.6 mm to (185.4, 1.34)
- moved R8 110.1 mm to (194.3, 1.71)
- moved C8 110.0 mm to (172.5, 19.4)
- moved U16 109.8 mm to (144.4, -4.92)
- moved C9 109.2 mm to (179.4, 10.8)
- moved D4 108.9 mm to (189.9, 1.75)
- moved U9 108.3 mm to (179.0, 3.05)
- moved C10 107.2 mm to (189.9, -1.27)
- moved D5 106.0 mm to (183.8, 7.79)
- moved R17 105.5 mm to (194.3, 4.66)
- moved D2 102.8 mm to (168.1, 19.4)
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- renumbered C21 to C13, C22 to C14, C27 to C17, C28 to C18, C29 to C19, C30 to C20, C31 to C21, C32 to C22, C33 to C23, J9 to J10, J10 to J11, J11 to J12, J12 to J13, J6 to J7, J7 to J8, J8 to J9, R9 to R13, R7 to R9
Connections:
- C10 pad 1: Net-(C10-Pad1) -> GND
- C10 pad 2: GND -> +3V3
- C15 pad 1: +3V3 -> GND
- C15 pad 2: GND -> +3V3
- C16 pad 1: +3V3 -> Net-(C16-Pad1)
- C7 pad 1: +3V3 -> Net-(C7-Pad1)
- C8 pad 1: +3V3 -> Net-(C8-Pad1)
- C9 pad 1: Net-(C9-Pad1) -> GND
- C9 pad 2: GND -> +3V3
- J2 pad 2: Net-(C10-Pad1) -> Net-(J2-Pad2)
- J3 pad 2: Net-(C12-Pad1) -> Net-(J3-Pad2)
- J4 pad 1: (no net) -> +5V
- J4 pad 2: Net-(C18-Pad1) -> /RELAY_MASTER
- J5 pad 2: Net-(C20-Pad1) -> Net-(J5-Pad2)
- R1 pad 2: Net-(C9-Pad1) -> Net-(C7-Pad1)
- R10 pad 1: Net-(F3-Pad1) -> GND
- R10 pad 2: Net-(C17-Pad1) -> Net-(D2-Pad1)
- R11 pad 1: Net-(F4-Pad1) -> GND
- R11 pad 2: Net-(C19-Pad1) -> Net-(R11-Pad2)
- R12 pad 2: /OUT2_EN -> Net-(R12-Pad2)
- R14 pad 1: GND -> Net-(F3-Pad1)
- R14 pad 2: Net-(D3-Pad1) -> Net-(C11-Pad1)
- R15 pad 1: GND -> Net-(F4-Pad1)
- R15 pad 2: Net-(D4-Pad1) -> Net-(C12-Pad1)
- R16 pad 1: Net-(F5-Pad1) -> Net-(R16-Pad1)
- R16 pad 2: Net-(C25-Pad1) -> /OUT2_EN
- R17 pad 1: GND -> Net-(R17-Pad1)
- R17 pad 2: /OUT4_EN -> /OUT3_EN
- R18 pad 2: Net-(D5-Pad1) -> Net-(R18-Pad2)
- R2 pad 2: Net-(C11-Pad1) -> Net-(C8-Pad1)
- R3 pad 1: GND -> Net-(R3-Pad1)
- R8 pad 2: Net-(D2-Pad1) -> Net-(R8-Pad2)
- U10 pad 7: Net-(C19-Pad1) -> Net-(C12-Pad1)
- U11 pad 1: Net-(C17-Pad1) -> Net-(J5-Pad2)
- U11 pad 2: /OUT2_EN -> Net-(J5-Pad2)
- U11 pad 3: +3V3 -> Net-(J5-Pad2)
- U11 pad 4: GND -> Net-(R16-Pad1)
- U11 pad 5: (no net) -> Net-(R22-Pad2)
- U11 pad 6: /OUT2_PG -> Net-(R18-Pad2)
- U11 pad 7: Net-(C18-Pad1) -> GND
- U12 pad 1: Net-(C19-Pad1) -> Net-(J6-Pad2)
- U12 pad 2: /OUT3_EN -> Net-(J6-Pad2)
- U12 pad 3: +3V3 -> Net-(J6-Pad2)
- U12 pad 4: GND -> Net-(R17-Pad1)
- U12 pad 5: (no net) -> Net-(R23-Pad2)
- U12 pad 6: /OUT3_PG -> Net-(R19-Pad2)
- U12 pad 7: Net-(C20-Pad1) -> GND
- U15 pad 7: Net-(C25-Pad1) -> Net-(C16-Pad1)
- U16 pad 1: Net-(C25-Pad1) -> Net-(J14-Pad2)
- U16 pad 2: /OUT4_EN -> Net-(J14-Pad2)
- U16 pad 3: +3V3 -> Net-(J14-Pad2)
- U16 pad 4: GND -> Net-(R25-Pad1)
- U16 pad 5: (no net) -> Net-(R28-Pad2)
- U16 pad 6: /OUT4_PG -> Net-(R26-Pad2)
- U16 pad 7: Net-(C26-Pad1) -> GND
- U2 pad 16: (no net) -> /RELAY_MASTER
- U2 pad 2: /OUT0_EN -> (no net)
- U2 pad 3: /OUT1_EN -> (no net)
- U2 pad 4: /OUT2_EN -> (no net)
- U2 pad 5: /OUT3_EN -> (no net)
- U2 pad 6: /OUT4_EN -> (no net)
- U3 pad 7: Net-(C9-Pad1) -> Net-(C7-Pad1)
- U4 pad 7: Net-(C11-Pad1) -> Net-(C8-Pad1)
- U5 pad 1: Net-(C9-Pad1) -> Net-(J2-Pad2)
- U5 pad 2: /OUT0_EN -> Net-(J2-Pad2)
- U5 pad 3: +3V3 -> Net-(J2-Pad2)
- U5 pad 4: GND -> Net-(R3-Pad1)
- U5 pad 5: (no net) -> Net-(R11-Pad2)
- U5 pad 6: /OUT0_PG -> Net-(R7-Pad2)
- U5 pad 7: Net-(C10-Pad1) -> GND
- U6 pad 1: Net-(C11-Pad1) -> Net-(J3-Pad2)
- U6 pad 2: /OUT1_EN -> Net-(J3-Pad2)
- U6 pad 3: +3V3 -> Net-(J3-Pad2)
- U6 pad 4: GND -> Net-(R4-Pad1)
- U6 pad 5: (no net) -> Net-(R12-Pad2)
- U6 pad 6: /OUT1_PG -> Net-(R8-Pad2)
- U6 pad 7: Net-(C12-Pad1) -> GND
- U8 pad 2: /OUT0_PG -> (no net)
- U8 pad 22: /OUT4_PG -> (no net)
- U8 pad 4: /OUT1_PG -> (no net)
- U8 pad 6: /OUT2_PG -> (no net)
- U8 pad 8: /OUT3_PG -> (no net)
- U9 pad 7: Net-(C17-Pad1) -> Net-(C11-Pad1)

Commit message: More progress on schematic and footprints
Parts:
- added D12: Red, LED_SMD:LED_0805_2012Metric, F.Cu at (201.9, -40.6)
- added D13: Red, LED_SMD:LED_0805_2012Metric, F.Cu at (185.5, -27.7)
- added D14: Red, LED_SMD:LED_0805_2012Metric, F.Cu at (201.9, -37.6)
- added D15: Red, LED_SMD:LED_0805_2012Metric, F.Cu at (190.0, -27.7)
- added D16: Red, LED_SMD:LED_0805_2012Metric, F.Cu at (185.5, -24.7)
- added F1: Fuse Holder BK-6013, BK-6013:BK-6013, F.Cu at (175.1, -38.9)
- added F2: Fuse Holder BK-6013, BK-6013:BK-6013, F.Cu at (175.1, -32.5)
- added F3: Fuse Holder BK-6013, BK-6013:BK-6013, F.Cu at (191.5, -38.9)
- added F4: Fuse Holder BK-6013, BK-6013:BK-6013, F.Cu at (175.1, -26.0)
- added F5: Fuse Holder BK-6013, BK-6013:BK-6013, F.Cu at (191.5, -32.5)
- added R29: 2k, Resistor_SMD:R_0805_2012Metric, F.Cu at (189.9, -24.7)
- added R30: 2k, Resistor_SMD:R_0805_2012Metric, F.Cu at (201.9, -34.6)
- added R31: 2k, Resistor_SMD:R_0805_2012Metric, F.Cu at (194.4, -27.8)
- added R32: 2k, Resistor_SMD:R_0805_2012Metric, F.Cu at (194.3, -24.7)
- added R33: 2k, Resistor_SMD:R_0805_2012Metric, F.Cu at (201.9, -31.7)
- D1, D2, D3, D4, D5: value LED_Small -> Red
- J1, J11, J12, J13, J14, J2, J3, J4, J5, J6, J7, J8, J9: footprint TerminalBlock:TerminalBlock_bornier-2_P5.08mm -> ScrewTerminals:EB147A-02-D
- J10: footprint TerminalBlock:TerminalBlock_bornier-3_P5.08mm -> ScrewTerminals:C72334_WJ500V-5.08-3P
- U2: value TPL7407LA -> TPL7407L
Connections:
- J14 pad 1: (no net) -> Net-(F5-Pad2)
- J2 pad 1: (no net) -> Net-(F1-Pad2)
- J3 pad 1: (no net) -> Net-(F2-Pad2)
- J5 pad 1: (no net) -> Net-(F3-Pad2)
- J6 pad 1: (no net) -> Net-(F4-Pad2)
- U8 pad 2: (no net) -> /OUT1_EN
- U8 pad 21: /OUT4_EN -> (no net)
- U8 pad 3: /OUT1_EN -> /OUT2_EN
- U8 pad 4: (no net) -> /OUT3_EN
- U8 pad 5: /OUT2_EN -> /OUT4_EN
- U8 pad 7: /OUT3_EN -> (no net)
