File: electronics/chainlinkDriverTester/chainlinkDriverTester.sch (KiCad schematic (older format))
At the start: 139 parts, among them J1 Inputs, J10 Sensor C, J11 Sensor D, J12 Motor E, J13 Motor F, J14 Sensor E, J15 Sensor F, J16 Power, J17 Power, J18 Power, J19 Outputs, J2 Inputs, J20 Outputs, J21 Outputs, J22 Power, J23 exp, J24 exp, J25 exp, J26 exp, J27 exp, J28 exp, J29 exp, J3 Motor A, J30 exp, J31 exp, J32 Conn_01x06_Female, J4 Inputs, J5 Motor B, J6 Motor C, J7 Motor D, J8 Sensor A, J9 Sensor B, U1 AP7361C-33E, U2 TTGO_TDisplay, U3 VN7007ALH, U4 MCP23017_SS, U5 INA219BxD, U6 MCP23017_SS

Commit message: Checkpoint
Parts:
- removed C8: 10uF, Capacitor_SMD:CP_Elec_4x5.3, symbol Device:CP_Small
- removed C9: 0.1uF, Capacitor_SMD:C_0805_2012Metric, symbol Device:C_Small
- removed J1, J2, J4: Inputs, ScrewTerminals:C8465_WJ500V-5.08-2P, symbol Connector:Screw_Terminal_01x02
- removed J16, J17, J18: Power, ScrewTerminals:C8465_WJ500V-5.08-2P, symbol Connector:Screw_Terminal_01x02
- removed J19, J20, J21: Outputs, ScrewTerminals:C8465_WJ500V-5.08-2P, symbol Connector:Screw_Terminal_01x02
- removed J23, J24, J25: exp, symbol Connector:Conn_01x04_Female
- removed R13, R14: 15k, Resistor_SMD:R_0805_2012Metric, symbol Device:R_Small
- removed U6: MCP23017_SS, Package_SO:SSOP-28_5.3x10.2mm_P0.65mm, symbol Interface_Expansion:MCP23017_SS
- added H10, H11, H12, H13, H14, H15, H16, H6, H7, H8, H9: MountingHole, MountingHole:MountingHole_3.2mm_M3_ISO7380_Pad, symbol Mechanical:MountingHole_Pad
- added TP69, TP70, TP71, TP72, TP73, TP74, TP75: TestPoint, TestPoint:TestPoint_THTPad_D2.0mm_Drill1.0mm, symbol Connector:TestPoint
- D3: footprint (none) -> Diode_SMD:D_SOD-123
- F1: footprint (none) -> Fuse:Fuse_0603_1608Metric
- J26, J27, J28, J29, J30, J31: footprint (none) -> Connector_PinHeader_2.54mm:PinHeader_1x04_P2.54mm_Vertical
- J32: footprint (none) -> Connector_PinSocket_2.54mm:PinSocket_1x06_P2.54mm_Vertical
- TP1, TP10, TP11, TP12, TP13, TP14, TP15, TP16, TP17, TP18, TP19, TP2, TP20, TP21, TP22, TP23, TP24, TP25, TP26, TP27, TP28, TP29, TP3, TP30, TP31, TP32, TP33, TP34, TP35, TP36, TP37, TP38, TP39, TP4, TP40, TP41, TP42, TP43, TP44, TP45, TP46, TP47, TP48, TP5, TP6, TP7, TP8, TP9: footprint (none) -> pogoPins:pogo1mm
- TP49, TP50, TP51, TP52, TP53, TP54, TP55, TP56, TP57, TP58, TP59, TP60, TP63, TP64, TP65, TP66, TP67, TP68: footprint (none) -> pogoPins:pogo2mm
- TP61, TP62: footprint (none) -> TestPoint:TestPoint_THTPad_D2.0mm_Drill1.0mm
Connections:
- net +3V3: now also TP75.1
- net +5V: now also TP73.1
- net SENSOR_A_GND: no longer U4.3 (GPB2)
- net SENSOR_A_VCC: no longer U4.2 (GPB1)
- net SENSOR_B_GND: no longer U4.6 (GPB5)
- net SENSOR_B_SIGNAL: now also U4.2 (GPB1); no longer U4.4 (GPB3)
- net SENSOR_B_VCC: no longer U4.5 (GPB4)
- net SENSOR_C_GND: no longer U4.21 (GPA0)
- net SENSOR_C_SIGNAL: now also U4.3 (GPB2); no longer U4.7 (GPB6)
- net SENSOR_C_VCC: no longer U4.8 (GPB7)
- net SENSOR_D_GND: no longer U4.24 (GPA3)
- net SENSOR_D_SIGNAL: now also U4.4 (GPB3); no longer U4.22 (GPA1)
- net SENSOR_D_VCC: no longer U4.23 (GPA2)
- net SENSOR_E_GND: no longer U4.27 (GPA6)
- net SENSOR_E_SIGNAL: now also U4.5 (GPB4); no longer U4.25 (GPA4)
- net SENSOR_E_VCC: no longer U4.26 (GPA5)
- net SENSOR_F_SIGNAL: now also U4.6 (GPB5); no longer U4.28 (GPA7)
- net at U2.23 (GPIO36): now also TP69.1
- net at U2.7 (GPIO15): now also TP71.1
- net at U2.9 (GPIO12): now also TP72.1
- net SW_IN: now reaches F2.1, U3.TAB (VCC)
- net at J26.1 (Pin_1): now also U4.21 (GPA0)
- net at J26.2 (Pin_2): now also U4.22 (GPA1)
- net at J26.3 (Pin_3): now also U4.23 (GPA2)
- net at J26.4 (Pin_4): now also U4.24 (GPA3)
- net at J29.1 (Pin_1): now also U4.25 (GPA4)
- net at J29.2 (Pin_2): now also U4.26 (GPA5)
- net at J29.3 (Pin_3): now also U4.27 (GPA6)
- net at J29.4 (Pin_4): now also U4.28 (GPA7)
- net at TP61.1: now also U4.7 (GPB6)
- net at TP62.1: now also U4.8 (GPB7)
- net at C4.2, C5.1, F1.2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: now also TP74.1
- net MCP_INT_0 renamed MCP_INT
- net MCP_INT_1: no longer names the net of U2.21 (GPIO38)
- net MCP_INT_1: now also TP70.1
- no-connect marks 28 -> 17
Other:
- note removed: "I2C ADDR: 0x21"
- moved on the sheet: C6, F1, J26, J27, J28, J29, J30, J31, R10, R4, TP61, TP62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

Commit message: Checkpoint. Placement done, starting routing
Parts:
- added D4: Red, LED_SMD:LED_0805_2012Metric, symbol Device:LED_Small
- added R13: 220, Resistor_SMD:R_0805_2012Metric, symbol Device:R_Small
Connections:
- net 3V3_FUSED: now also D4.2 (A)
- net GND: now also R13.1
- net SENSOR_D_SIGNAL: now also U4.6 (GPB5); no longer U4.4 (GPB3)
- net SENSOR_E_SIGNAL: now also U4.7 (GPB6); no longer U4.5 (GPB4)
- net SENSOR_F_SIGNAL: now also U4.8 (GPB7); no longer U4.6 (GPB5)
- net at TP61.1: now also U4.4 (GPB3); no longer U4.7 (GPB6)
- net at TP62.1: now also U4.5 (GPB4); no longer U4.8 (GPB7)
- new net: D4.1 (K), R13.2
Other:
- moved on the sheet: TP61, TP62
Changed lines of the file:
@@
 	7650 1100 7800 1100
 Wire Wire Line
-	9050 1100 9800 1100
+	9050 1100 9300 1100
 Text Label 9800 1100 2    50   ~ 0
 3V3_FUSED
@@
 L Connector:TestPoint TP62
 U 1 1 61F7F830
-P 8550 6400
-F 0 "TP62" V 8550 6588 50  0000 L CNN
-F 1 "TestPoint" V 8595 6588 50  0001 L CNN
-F 2 "TestPoint:TestPoint_THTPad_D2.0mm_Drill1.0mm" H 8750 6400 50  0001 C CNN
-F 3 "~" H 8750 6400 50  0001 C CNN
-	1    8550 6400
+P 8550 6100
+F 0 "TP62" V 8550 6288 50  0000 L CNN
+F 1 "TestPoint" V 8595 6288 50  0001 L CNN
+F 2 "TestPoint:TestPoint_THTPad_D2.0mm_Drill1.0mm" H 8750 6100 50  0001 C CNN
+F 3 "~" H 8750 6100 50  0001 C CNN
+	1    8550 6100
 	0    1    1    0
 $EndComp
@@
 L Connector:TestPoint TP61
 U 1 1 61F7E6FB
-P 8550 6300
-F 0 "TP61" V 8550 6488 50  0000 L CNN
-F 1 "TestPoint" V 8595 6488 50  0001 L CNN
-F 2 "TestPoint:TestPoint_THTPad_D2.0mm_Drill1.0mm" H 8750 6300 50  0001 C CNN
-F 3 "~" H 8750 6300 50  0001 C CNN
-	1    8550 6300
+P 8550 6000
+F 0 "TP61" V 8550 6188 50  0000 L CNN
+F 1 "TestPoint" V 8595 6188 50  0001 L CNN
+F 2 "TestPoint:TestPoint_THTPad_D2.0mm_Drill1.0mm" H 8750 6000 50  0001 C CNN
+F 3 "~" H 8750 6000 50  0001 C CNN
+	1    8550 6000
 	0    1    1    0
 $EndComp
@@
 	1    0    0    -1
 $EndComp
+Text Label 9550 6400 2    50   ~ 0
+SENSOR_F_SIGNAL
+Text Label 9550 6300 2    50   ~ 0
+SENSOR_E_SIGNAL
 Text Label 9550 6200 2    50   ~ 0
-SENSOR_F_SIGNAL
-Text Label 9550 6100 2    50   ~ 0
-SENSOR_E_SIGNAL
-Text Label 9550 6000 2    50   ~ 0
 SENSOR_D_SIGNAL
 Text Label 9550 5900 2    50   ~ 0
@@
 	8550 5900 9550 5900
 Wire Wire Line
-	8550 6000 9550 6000
-Wire Wire Line
-	8550 6100 9550 6100
-Wire Wire Line
 	8550 6200 9550 6200
+Wire Wire Line
+	8550 6300 9550 6300
+Wire Wire Line
+	8550 6400 9550 6400
 $Comp
 L Mechanical:MountingHole_Pad H10
@@
 Text Label 14500 4300 0    50   ~ 0
 SW_IN
+$Comp
+L Device:LED_Small D?
+U 1 1 607210C0
+P 9300 1200
+AR Path="/60D00052/607210C0" Ref="D?"  Part="1"
+AR Path="/607210C0" Ref="D4"  Part="1"
+F 0 "D4" V 9350 1350 50  0000 R CNN
+F 1 "Red" V 9250 1400 50  0000 R CNN
+F 2 "LED_SMD:LED_0805_2012Metric" V 9300 1200 50  0001 C CNN
+F 3 "~" V 9300 1200 50  0001 C CNN
+	1    9300 1200
+	0    -1   -1   0
+$EndComp
+$Comp
+L Device:R_Small R?
+U 1 1 6072153E
+P 9300 1450
+AR Path="/60D00052/6072153E" Ref="R?"  Part="1"
+AR Path="/6072153E" Ref="R13"  Part="1"
+F 0 "R13" H 9400 1400 50  0000 C CNN
+F 1 "220" H 9400 1500 50  0000 C CNN
+F 2 "Resistor_SMD:R_0805_2012Metric" H 9300 1450 50  0001 C CNN
+F 3 "~" H 9300 1450 50  0001 C CNN
+	1    9300 1450
+	-1   0    0    1
+$EndComp
+Wire Wire Line
+	9300 1300 9300 1350
+Wire Wire Line
+	9300 1550 9300 1650
+Connection ~ 9300 1100
+Wire Wire Line
+	9300 1100 9800 1100
+$Comp
+L power:GND #PWR02
+U 1 1 6074C1AB
+P 9300 1650
+F 0 "#PWR02" H 9300 1400 50  0001 C CNN
+F 1 "GND" H 9305 1477 50  0000 C CNN
+F 2 "" H 9300 1650 50  0001 C CNN
+F 3 "" H 9300 1650 50  0001 C CNN
+	1    9300 1650
+	1    0    0    -1
+$EndComp
 $EndSCHEMATC

Commit message: Finished routing
Parts:
- removed TP72: TestPoint, TestPoint:TestPoint_THTPad_D2.0mm_Drill1.0mm, symbol Connector:TestPoint
- added C10, C8, C9: 0.1uF, Capacitor_SMD:C_0805_2012Metric, symbol Device:C_Small
- added D5, D6: WS2812B, LED_SMD:LED_WS2812B_PLCC4_5.0x5.0mm_P3.2mm, symbol LED:WS2812B
- added U6: SN74LV1T34DBV, Package_TO_SOT_SMD:SOT-23-5, symbol Logic_LevelTranslator:SN74LV1T34DBV
Connections:
- net +3V3: no longer U2.12 (3V3)
- net +5V: now also C10.1, C8.1, C9.1, D5.1 (VDD), D6.1 (VDD), U6.5 (VCC)
- net GND: now also C10.2, C8.2, C9.2, D5.3 (VSS), D6.3 (VSS), U6.3 (GND)
- net LED: now reaches U2.9 (GPIO12)
- net LED: now also U6.2 (A)
- new net: D5.4 (DIN), U6.4 (Y)
- new net: D5.2 (DOUT), D6.4 (DIN)
- no-connect marks 17 -> 19
Changed lines of the file:
@@
 Wire Wire Line
 	3750 4100 3600 4100
-Wire Wire Line
-	2100 5050 2100 5200
-Wire Wire Line
-	2100 5200 2600 5200
 $Comp
 L power:+3.3V #PWR0105
@@
 F 3 "" H 3750 4000 50  0001 C CNN
 	1    3750 4000
-	1    0    0    -1
-$EndComp
-$Comp
-L power:+3.3V #PWR0106
-U 1 1 60D0A520
-P 2100 5050
-F 0 "#PWR0106" H 2100 4900 50  0001 C CNN
-F 1 "+3.3V" H 2115 5223 50  0000 C CNN
-F 2 "" H 2100 5050 50  0001 C CNN
-F 3 "" H 2100 5050 50  0001 C CNN
-	1    2100 5050
 	1    0    0    -1
 $EndComp
@@
 	0    1    1    0
 $EndComp
-$Comp
-L Connector:TestPoint TP71
-U 1 1 62B8767D
-P 2600 4700
-F 0 "TP71" V 2600 4950 50  0000 C CNN
-F 1 "TestPoint" V 2704 4772 50  0001 C CNN
-F 2 "TestPoint:TestPoint_THTPad_D2.0mm_Drill1.0mm" H 2800 4700 50  0001 C CNN
-F 3 "~" H 2800 4700 50  0001 C CNN
-	1    2600 4700
-	0    -1   -1   0
-$EndComp
-$Comp
-L Connector:TestPoint TP72
-U 1 1 62B87DD9
-P 2600 4900
-F 0 "TP72" V 2600 5150 50  0000 C CNN
-F 1 "TestPoint" V 2704 4972 50  0001 C CNN
-F 2 "TestPoint:TestPoint_THTPad_D2.0mm_Drill1.0mm" H 2800 4900 50  0001 C CNN
-F 3 "~" H 2800 4900 50  0001 C CNN
-	1    2600 4900
-	0    -1   -1   0
-$EndComp
 Wire Wire Line
 	8200 1100 8850 1100
@@
 	1    0    0    -1
 $EndComp
+$Comp
+L Logic_LevelTranslator:SN74LV1T34DBV U6
+U 1 1 6077F65C
+P 6550 8900
+F 0 "U6" H 6894 8946 50  0000 L CNN
+F 1 "SN74LV1T34DBV" H 6894 8855 50  0000 L CNN
+F 2 "Package_TO_SOT_SMD:SOT-23-5" H 7200 8650 50  0001 C CNN
+F 3 "https://www.ti.com/lit/ds/symlink/sn74lv1t34.pdf" H 6150 8700 50  0001 C CNN
+	1    6550 8900
+	1    0    0    -1
+$EndComp
+$Comp
+L LED:WS2812B D5
+U 1 1 60781C6E
+P 7400 8900
+F 0 "D5" H 7744 8946 50  0000 L CNN
+F 1 "WS2812B" H 7744 8855 50  0000 L CNN
+F 2 "LED_SMD:LED_WS2812B_PLCC4_5.0x5.0mm_P3.2mm" H 7450 8600 50  0001 L TNN
+F 3 "https://cdn-shop.adafruit.com/datasheets/WS2812B.pdf" H 7500 8525 50  0001 L TNN
+	1    7400 8900
+	1    0    0    -1
+$EndComp
+Wire Wire Line
+	6850 8900 7100 8900
+$Comp
+L power:+5V #PWR03
+U 1 1 6079EC4F
+P 6950 8450
+F 0 "#PWR03" H 6950 8300 50  0001 C CNN
+F 1 "+5V" H 6965 8623 50  0000 C CNN
+F 2 "" H 6950 8450 50  0001 C CNN
+F 3 "" H 6950 8450 50  0001 C CNN
+	1    6950 8450
+	1    0    0    -1
+$EndComp
+$Comp
+L power:GND #PWR05
+U 1 1 6079F756
+P 6950 9300
+F 0 "#PWR05" H 6950 9050 50  0001 C CNN
+F 1 "GND" H 6955 9127 50  0000 C CNN
+F 2 "" H 6950 9300 50  0001 C CNN
+F 3 "" H 6950 9300 50  0001 C CNN
+	1    6950 9300
+	1    0    0    -1
+$EndComp
+Wire Wire Line
+	6550 9200 6950 9200
+Wire Wire Line
+	6950 9300 6950 9200
+Connection ~ 6950 9200
+Wire Wire Line
+	6950 9200 7050 9200
+Wire Wire Line
+	6550 8600 6950 8600
+Wire Wire Line
+	6950 8450 6950 8600
+Connection ~ 6950 8600
+Wire Wire Line
+	6950 8600 7050 8600
+Wire Wire Line
+	6250 8900 5600 8900
+Text Label 5600 8900 0    50   ~ 0
+LED
+$Comp
+L Connector:TestPoint TP71
+U 1 1 62B8767D
+P 2600 4700
+F 0 "TP71" V 2600 4950 50  0000 C CNN
+F 1 "TestPoint" V 2704 4772 50  0001 C CNN
+F 2 "TestPoint:TestPoint_THTPad_D2.0mm_Drill1.0mm" H 2800 4700 50  0001 C CNN
+F 3 "~" H 2800 4700 50  0001 C CNN
+	1    2600 4700
+	0    -1   -1   0
+$EndComp
+Wire Wire Line
+	1900 4900 2600 4900
+Text Label 1900 4900 0    50   ~ 0
+LED
+$Comp
+L LED:WS2812B D6
+U 1 1 60898405
+P 8200 8900
+F 0 "D6" H 8544 8946 50  0000 L CNN
+F 1 "WS2812B" H 8544 8855 50  0000 L CNN
+F 2 "LED_SMD:LED_WS2812B_PLCC4_5.0x5.0mm_P3.2mm" H 8250 8600 50  0001 L TNN
+F 3 "https://cdn-shop.adafruit.com/datasheets/WS2812B.pdf" H 8300 8525 50  0001 L TNN
+	1    8200 8900
+	1    0    0    -1
+$EndComp
+Wire Wire Line
+	7400 8600 7850 8600
+Connection ~ 7400 8600
+Connection ~ 7400 9200
+Wire Wire Line
+	7700 8900 7900 8900
+$Comp
+L Device:C_Small C?
+U 1 1 608F3043
+P 6200 8700
+AR Path="/60D00052/608F3043" Ref="C?"  Part="1"
+AR Path="/608F3043" Ref="C9"  Part="1"
+F 0 "C9" H 6250 8950 50  0000 R CNN
+F 1 "0.1uF" H 6300 8850 50  0000 R CNN
+F 2 "Capacitor_SMD:C_0805_2012Metric" H 6200 8700 50  0001 C CNN
+F 3 "~" H 6200 8700 50  0001 C CNN
+	1    6200 8700
+	1    0    0    -1
+$EndComp
+Wire Wire Line
+	6200 8600 6550 8600
+Connection ~ 6550 8600
+Wire Wire Line
+	6200 8800 6200 9200
+Wire Wire Line
+	6200 9200 6550 9200
+Connection ~ 6550 9200
+$Comp
+L Device:C_Small C?
+U 1 1 60932510
+P 7050 8700
+AR Path="/60D00052/60932510" Ref="C?"  Part="1"
+AR Path="/60932510" Ref="C10"  Part="1"
+F 0 "C10" H 7100 8950 50  0000 R CNN
+F 1 "0.1uF" H 7150 8850 50  0000 R CNN
+F 2 "Capacitor_SMD:C_0805_2012Metric" H 7050 8700 50  0001 C CNN
+F 3 "~" H 7050 8700 50  0001 C CNN
+	1    7050 8700
+	1    0    0    -1
+$EndComp
+Connection ~ 7050 8600
+Wire Wire Line
+	7050 8600 7400 8600
+Wire Wire Line
+	7050 8800 7050 9200
+Connection ~ 7050 9200
+Wire Wire Line
+	7050 9200 7400 9200
+$Comp
+L Device:C_Small C?
+U 1 1 60952141
+P 7850 8700
+AR Path="/60D00052/60952141" Ref="C?"  Part="1"
+AR Path="/60952141" Ref="C8"  Part="1"
+F 0 "C8" H 7900 8950 50  0000 R CNN
+F 1 "0.1uF" H 7950 8850 50  0000 R CNN
+F 2 "Capacitor_SMD:C_0805_2012Metric" H 7850 8700 50  0001 C CNN
+F 3 "~" H 7850 8700 50  0001 C CNN
+	1    7850 8700
+	1    0    0    -1
+$EndComp
+NoConn ~ 8500 8900
+Wire Wire Line
+	7400 9200 7850 9200
+Connection ~ 7850 8600
+Wire Wire Line
+	7850 8600 8200 8600
+Wire Wire Line
+	7850 8800 7850 9200
+Connection ~ 7850 9200
+Wire Wire Line
+	7850 9200 8200 9200
+NoConn ~ 2600 5200
 $EndSCHEMATC
