File: electronics/sensor_smd/sensor_smd.kicad_sch (KiCad schematic)
At the start: 7 parts, among them J1 HEADER MALE RA, U1 HX6286

Commit message: Clean up classic, clean up readme, start setting up panelization and export for sensor_smd
Parts:
- D1: LCSC (none) -> C2286
- H1, H2, J1, JP1: now left out of the parts list
- R1: LCSC (none) -> C21190
- U1: LCSC (none) -> C495736
Changed lines of the file:
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@@
   )
   (symbol (lib_id "Jumper:Jumper_2_Bridged") (at 95.25 29.21 0) (unit 1)
-    (in_bom yes) (on_board yes) (fields_autoplaced)
+    (in_bom no) (on_board yes) (fields_autoplaced)
     (property "Reference" "JP1" (id 0) (at 95.25 22.86 0))
     (property "Value" "LED enable" (id 1) (at 95.25 25.4 0))
@@
       (effects (font (size 1.27 1.27) italic) (justify left) hide)
     )
-    (property "Datasheet" "https://www.allegromicro.com/-/media/files/datasheets/a110x-datasheet.ashx" (id 3) (at 90.17 26.67 0)
+    (property "Datasheet" "" (id 3) (at 90.17 26.67 0)
+      (effects (font (size 1.27 1.27)) hide)
+    )
+    (property "LCSC" "C495736" (id 4) (at 90.17 43.18 0)
       (effects (font (size 1.27 1.27)) hide)
     )
@@
   )
   (symbol (lib_id "Mechanical:MountingHole") (at 156.21 33.02 0) (unit 1)
-    (in_bom yes) (on_board yes) (fields_autoplaced)
+    (in_bom no) (on_board yes) (fields_autoplaced)
     (property "Reference" "H1" (id 0) (at 158.75 31.7499 0)
       (effects (font (size 1.27 1.27)) (justify left))
@@
   )
   (symbol (lib_id "Mechanical:MountingHole") (at 156.21 39.37 0) (unit 1)
-    (in_bom yes) (on_board yes) (fields_autoplaced)
+    (in_bom no) (on_board yes) (fields_autoplaced)
     (property "Reference" "H2" (id 0) (at 158.75 38.0999 0)
       (effects (font (size 1.27 1.27)) (justify left))
@@
   )
   (symbol (lib_id "Connector:Conn_01x03_Male") (at 29.21 44.45 0) (unit 1)
-    (in_bom yes) (on_board yes) (fields_autoplaced)
+    (in_bom no) (on_board yes) (fields_autoplaced)
     (property "Reference" "J1" (id 0) (at 29.845 36.83 0))
     (property "Value" "HEADER MALE RA" (id 1) (at 29.845 39.37 0))
@@
       (effects (font (size 1.27 1.27)) hide)
     )
+    (property "LCSC" "C2286" (id 4) (at 101.6 39.37 90)
+      (effects (font (size 1.27 1.27)) hide)
+    )
     (pin "1")
     (pin "2")
@@
       (effects (font (size 1.27 1.27)) hide)
     )
+    (property "LCSC" "C21190" (id 4) (at 101.6 33.02 0)
+      (effects (font (size 1.27 1.27)) hide)
+    )

Commit message: Remove H2 from placement, rotate sensor
Parts:
- U1: JLCPCB_CORRECTION (none) -> 0; 0; 180
Changed lines of the file:
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@@
+      (effects (font (size 1.27 1.27)) hide)
+    )
+    (property "JLCPCB_CORRECTION" "0; 0; 180" (id 5) (at 90.17 43.18 0)
       (effects (font (size 1.27 1.27)) hide)
     )
