File: electronics/sensor_smd/sensor_smd.kicad_sch (KiCad schematic)
At the start: 7 parts, among them J1 HEADER MALE RA, U1 HX6286

Commit message: Updates
Other:
- title: (none) -> splitflap sensor smd
Changed lines of the file:
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@@
 (kicad_sch (version 20211123) (generator eeschema)
-  (paper "A5")
+  (paper "User" 150.012 119.99)
+  (title_block
+    (title "splitflap sensor smd")
+  )
   (junction (at 101.6 43.18) (diameter 0) (color 0 0 0 0)
   )
