File: electronics/chainlinkDriver/chainlinkDriver.sch (KiCad schematic (older format))
At the start: 65 parts, among them J10 Sensor, J11 Sensor, J12 Motor, J13 Motor, J14 Sensor, J15 Sensor, J16 Power, J17 Power, J18 Power, J19 IDC, J20 IDC, J3 Motor, J5 Motor, J6 Motor, J7 Motor, J8 Sensor, J9 Sensor, U1 74HC595, U10 TPL7407L, U2 TPL7407L, U3 74HC125, U4 74HC165, U5 74HC595, U6 TPL7407L, U7 74HC595, U8 TPL7407L, U9 74HC595

Commit message: WIP updating parts for assembly
Parts:
- J10, J11, J14, J15, J8, J9: LCSC (none) -> C49257
- J12, J13, J3, J5, J6, J7: LCSC (none) -> C157991
- J19, J20: LCSC (none) -> C9135
Changed lines of the file:
@@
 F 2 "Connector_JST:JST_XH_B5B-XH-A_1x05_P2.50mm_Vertical" H 1700 2700 50  0001 C CNN
 F 3 "~" H 1700 2700 50  0001 C CNN
+F 4 "C157991" H 1672 2723 50  0001 C CNN "LCSC"
 	1    1700 2700
 	-1   0    0    -1
@@
 F 2 "Connector_JST:JST_XH_B5B-XH-A_1x05_P2.50mm_Vertical" H 3100 2700 50  0001 C CNN
 F 3 "~" H 3100 2700 50  0001 C CNN
+F 4 "C157991" H 3072 2723 50  0001 C CNN "LCSC"
 	1    3100 2700
 	-1   0    0    -1
@@
 F 2 "Connector_JST:JST_XH_B5B-XH-A_1x05_P2.50mm_Vertical" H 4500 2700 50  0001 C CNN
 F 3 "~" H 4500 2700 50  0001 C CNN
+F 4 "C157991" H 4472 2723 50  0001 C CNN "LCSC"
 	1    4500 2700
 	-1   0    0    -1
@@
 F 2 "Connector_JST:JST_XH_B5B-XH-A_1x05_P2.50mm_Vertical" H 5900 2700 50  0001 C CNN
 F 3 "~" H 5900 2700 50  0001 C CNN
+F 4 "C157991" H 5872 2723 50  0001 C CNN "LCSC"
 	1    5900 2700
 	-1   0    0    -1
@@
 F 2 "Connector_PinHeader_2.54mm:PinHeader_1x03_P2.54mm_Vertical" H 14950 2350 50  0001 C CNN
 F 3 "~" H 14950 2350 50  0001 C CNN
+F 4 "C49257" H 14922 2373 50  0001 C CNN "LCSC"
 	1    14950 2350
 	-1   0    0    1
@@
 F 2 "Connector_PinHeader_2.54mm:PinHeader_1x03_P2.54mm_Vertical" H 14950 2750 50  0001 C CNN
 F 3 "~" H 14950 2750 50  0001 C CNN
+F 4 "C49257" H 14922 2773 50  0001 C CNN "LCSC"
 	1    14950 2750
 	-1   0    0    1
@@
 F 2 "Connector_PinHeader_2.54mm:PinHeader_1x03_P2.54mm_Vertical" H 14950 3150 50  0001 C CNN
 F 3 "~" H 14950 3150 50  0001 C CNN
+F 4 "C49257" H 14922 3173 50  0001 C CNN "LCSC"
 	1    14950 3150
 	-1   0    0    1
@@
 F 2 "Connector_PinHeader_2.54mm:PinHeader_1x03_P2.54mm_Vertical" H 14950 3550 50  0001 C CNN
 F 3 "~" H 14950 3550 50  0001 C CNN
+F 4 "C49257" H 14922 3573 50  0001 C CNN "LCSC"
 	1    14950 3550
 	-1   0    0    1
@@
 F 2 "Connector_JST:JST_XH_B5B-XH-A_1x05_P2.50mm_Vertical" H 7250 2700 50  0001 C CNN
 F 3 "~" H 7250 2700 50  0001 C CNN
+F 4 "C157991" H 7222 2723 50  0001 C CNN "LCSC"
 	1    7250 2700
 	-1   0    0    -1
@@
 F 2 "Connector_JST:JST_XH_B5B-XH-A_1x05_P2.50mm_Vertical" H 8650 2700 50  0001 C CNN
 F 3 "~" H 8650 2700 50  0001 C CNN
+F 4 "C157991" H 8622 2723 50  0001 C CNN "LCSC"
 	1    8650 2700
 	-1   0    0    -1
@@
 F 2 "Connector_PinHeader_2.54mm:PinHeader_1x03_P2.54mm_Vertical" H 14950 3950 50  0001 C CNN
 F 3 "~" H 14950 3950 50  0001 C CNN
+F 4 "C49257" H 14922 3973 50  0001 C CNN "LCSC"
 	1    14950 3950
 	-1   0    0    1
@@
 F 2 "Connector_PinHeader_2.54mm:PinHeader_1x03_P2.54mm_Vertical" H 14950 4350 50  0001 C CNN
 F 3 "~" H 14950 4350 50  0001 C CNN
+F 4 "C49257" H 14922 4373 50  0001 C CNN "LCSC"
 	1    14950 4350
 	-1   0    0    1
@@
 F 2 "ModifiedSymbols:IDC-Header_2x04_P2.54mm_Vertical" H 2250 6500 50  0001 C CNN
 F 3 "~" H 2250 6500 50  0001 C CNN
+F 4 "C9135" H 2300 6726 50  0001 C CNN "LCSC"
 	1    2250 6500
 	1    0    0    -1
@@
 F 2 "ModifiedSymbols:IDC-Header_2x04_P2.54mm_Vertical" H 3850 6500 50  0001 C CNN
 F 3 "~" H 3850 6500 50  0001 C CNN
+F 4 "C9135" H 3900 6726 50  0001 C CNN "LCSC"
 	1    3850 6500
 	1    0    0    -1

Commit message: More placement updates
Parts:
- C8: JLCPCB_CORRECTION 0;0;180 -> (none); LCSC C134721 -> C176661; LCSC_ALT_3V3_CAP C176661 -> (none)
- J10, J11, J14, J15, J8, J9: JLCPCB_CORRECTION (none) -> 2.54;0;-90
- J12, J13, J3, J5, J6, J7: JLCPCB_CORRECTION (none) -> -5;0;-90
- J16, J17, J18: JLCPCB_CORRECTION 2.40;0;0 -> -2.40;0;180
- J19, J20: JLCPCB_CORRECTION (none) -> 1.27;3.81;-90
Changed lines of the file:
@@
 F 3 "~" H 1700 2700 50  0001 C CNN
 F 4 "C157991" H 1672 2723 50  0001 C CNN "LCSC"
+F 5 "-5;0;-90" H 1672 2723 50  0001 C CNN "JLCPCB_CORRECTION"
 	1    1700 2700
 	-1   0    0    -1
@@
 F 3 "~" H 3100 2700 50  0001 C CNN
 F 4 "C157991" H 3072 2723 50  0001 C CNN "LCSC"
+F 5 "-5;0;-90" H 3072 2723 50  0001 C CNN "JLCPCB_CORRECTION"
 	1    3100 2700
 	-1   0    0    -1
@@
 F 3 "~" H 4500 2700 50  0001 C CNN
 F 4 "C157991" H 4472 2723 50  0001 C CNN "LCSC"
+F 5 "-5;0;-90" H 4472 2723 50  0001 C CNN "JLCPCB_CORRECTION"
 	1    4500 2700
 	-1   0    0    -1
@@
 F 3 "~" H 5900 2700 50  0001 C CNN
 F 4 "C157991" H 5872 2723 50  0001 C CNN "LCSC"
+F 5 "-5;0;-90" H 5872 2723 50  0001 C CNN "JLCPCB_CORRECTION"
 	1    5900 2700
 	-1   0    0    -1
@@
 F 3 "~" H 14950 2350 50  0001 C CNN
 F 4 "C49257" H 14922 2373 50  0001 C CNN "LCSC"
+F 5 "2.54;0;-90" H 14922 2373 50  0001 C CNN "JLCPCB_CORRECTION"
 	1    14950 2350
 	-1   0    0    1
@@
 F 3 "~" H 14950 2750 50  0001 C CNN
 F 4 "C49257" H 14922 2773 50  0001 C CNN "LCSC"
+F 5 "2.54;0;-90" H 14922 2773 50  0001 C CNN "JLCPCB_CORRECTION"
 	1    14950 2750
 	-1   0    0    1
@@
 F 3 "~" H 14950 3150 50  0001 C CNN
 F 4 "C49257" H 14922 3173 50  0001 C CNN "LCSC"
+F 5 "2.54;0;-90" H 14922 3173 50  0001 C CNN "JLCPCB_CORRECTION"
 	1    14950 3150
 	-1   0    0    1
@@
 F 3 "~" H 14950 3550 50  0001 C CNN
 F 4 "C49257" H 14922 3573 50  0001 C CNN "LCSC"
+F 5 "2.54;0;-90" H 14922 3573 50  0001 C CNN "JLCPCB_CORRECTION"
 	1    14950 3550
 	-1   0    0    1
@@
 F 3 "~" H 7250 2700 50  0001 C CNN
 F 4 "C157991" H 7222 2723 50  0001 C CNN "LCSC"
+F 5 "-5;0;-90" H 7222 2723 50  0001 C CNN "JLCPCB_CORRECTION"
 	1    7250 2700
 	-1   0    0    -1
@@
 F 3 "~" H 8650 2700 50  0001 C CNN
 F 4 "C157991" H 8622 2723 50  0001 C CNN "LCSC"
+F 5 "-5;0;-90" H 8622 2723 50  0001 C CNN "JLCPCB_CORRECTION"
 	1    8650 2700
 	-1   0    0    -1
@@
 F 3 "~" H 14950 3950 50  0001 C CNN
 F 4 "C49257" H 14922 3973 50  0001 C CNN "LCSC"
+F 5 "2.54;0;-90" H 14922 3973 50  0001 C CNN "JLCPCB_CORRECTION"
 	1    14950 3950
 	-1   0    0    1
@@
 F 3 "~" H 14950 4350 50  0001 C CNN
 F 4 "C49257" H 14922 4373 50  0001 C CNN "LCSC"
+F 5 "2.54;0;-90" H 14922 4373 50  0001 C CNN "JLCPCB_CORRECTION"
 	1    14950 4350
 	-1   0    0    1
@@
 F 4 "C8465" H 1600 900 50  0001 C CNN "LCSC"
 F 5 "C395868" H 1600 900 50  0001 C CNN "LCSC_ALT_SCREW_DIBO"
-F 6 "2.40;0;0" H 1600 900 50  0001 C CNN "JLCPCB_CORRECTION"
+F 6 "-2.40;0;180" H 1600 900 50  0001 C CNN "JLCPCB_CORRECTION"
 	1    1600 900
 	1    0    0    -1
@@
 F 4 "C8465" H 1600 1100 50  0001 C CNN "LCSC"
 F 5 "C395868" H 1600 1100 50  0001 C CNN "LCSC_ALT_SCREW_DIBO"
-F 6 "2.40;0;0" H 1600 1100 50  0001 C CNN "JLCPCB_CORRECTION"
+F 6 "-2.40;0;180" H 1600 1100 50  0001 C CNN "JLCPCB_CORRECTION"
 	1    1600 1100
 	1    0    0    -1
@@
 F 4 "C8465" H 1600 1300 50  0001 C CNN "LCSC"
 F 5 "C395868" H 1600 1300 50  0001 C CNN "LCSC_ALT_SCREW_DIBO"
-F 6 "2.40;0;0" H 1600 1300 50  0001 C CNN "JLCPCB_CORRECTION"
+F 6 "-2.40;0;180" H 1600 1300 50  0001 C CNN "JLCPCB_CORRECTION"
 	1    1600 1300
 	1    0    0    -1
@@
 F 3 "~" H 2250 6500 50  0001 C CNN
 F 4 "C9135" H 2300 6726 50  0001 C CNN "LCSC"
+F 5 "1.27;3.81;-90" H 2300 6726 50  0001 C CNN "JLCPCB_CORRECTION"
 	1    2250 6500
 	1    0    0    -1
@@
 F 3 "~" H 3850 6500 50  0001 C CNN
 F 4 "C9135" H 3900 6726 50  0001 C CNN "LCSC"
+F 5 "1.27;3.81;-90" H 3900 6726 50  0001 C CNN "JLCPCB_CORRECTION"
 	1    3850 6500
 	1    0    0    -1
@@
 F 2 "Capacitor_SMD:CP_Elec_4x5.3" H 3500 1050 50  0001 C CNN
 F 3 "~" H 3500 1050 50  0001 C CNN
-F 4 "C134721" H 3500 1050 50  0001 C CNN "LCSC"
-F 5 "0;0;180" H 3500 1050 50  0001 C CNN "JLCPCB_CORRECTION"
-F 6 "C176661" H 3500 1050 50  0001 C CNN "LCSC_ALT_3V3_CAP"
+F 4 "C176661" H 3500 1050 50  0001 C CNN "LCSC"
 	1    3500 1050
 	1    0    0    -1

Commit message: More updates
Parts:
- J10, J11, J14, J15, J8, J9: JLCPCB_CORRECTION 2.54;0;-90 -> 0;2.54;-90
- J12, J13, J3, J5, J6, J7: JLCPCB_CORRECTION -5;0;-90 -> -5;0;-180
- J16, J17, J18: JLCPCB_CORRECTION -2.40;0;180 -> 2.40;0;180
Changed lines of the file:
@@
 F 3 "~" H 1700 2700 50  0001 C CNN
 F 4 "C157991" H 1672 2723 50  0001 C CNN "LCSC"
-F 5 "-5;0;-90" H 1672 2723 50  0001 C CNN "JLCPCB_CORRECTION"
+F 5 "-5;0;-180" H 1672 2723 50  0001 C CNN "JLCPCB_CORRECTION"
 	1    1700 2700
 	-1   0    0    -1
@@
 F 3 "~" H 3100 2700 50  0001 C CNN
 F 4 "C157991" H 3072 2723 50  0001 C CNN "LCSC"
-F 5 "-5;0;-90" H 3072 2723 50  0001 C CNN "JLCPCB_CORRECTION"
+F 5 "-5;0;-180" H 3072 2723 50  0001 C CNN "JLCPCB_CORRECTION"
 	1    3100 2700
 	-1   0    0    -1
@@
 F 3 "~" H 4500 2700 50  0001 C CNN
 F 4 "C157991" H 4472 2723 50  0001 C CNN "LCSC"
-F 5 "-5;0;-90" H 4472 2723 50  0001 C CNN "JLCPCB_CORRECTION"
+F 5 "-5;0;-180" H 4472 2723 50  0001 C CNN "JLCPCB_CORRECTION"
 	1    4500 2700
 	-1   0    0    -1
@@
 F 3 "~" H 5900 2700 50  0001 C CNN
 F 4 "C157991" H 5872 2723 50  0001 C CNN "LCSC"
-F 5 "-5;0;-90" H 5872 2723 50  0001 C CNN "JLCPCB_CORRECTION"
+F 5 "-5;0;-180" H 5872 2723 50  0001 C CNN "JLCPCB_CORRECTION"
 	1    5900 2700
 	-1   0    0    -1
@@
 F 3 "~" H 14950 2350 50  0001 C CNN
 F 4 "C49257" H 14922 2373 50  0001 C CNN "LCSC"
-F 5 "2.54;0;-90" H 14922 2373 50  0001 C CNN "JLCPCB_CORRECTION"
+F 5 "0;2.54;-90" H 14922 2373 50  0001 C CNN "JLCPCB_CORRECTION"
 	1    14950 2350
 	-1   0    0    1
@@
 F 3 "~" H 14950 2750 50  0001 C CNN
 F 4 "C49257" H 14922 2773 50  0001 C CNN "LCSC"
-F 5 "2.54;0;-90" H 14922 2773 50  0001 C CNN "JLCPCB_CORRECTION"
+F 5 "0;2.54;-90" H 14922 2773 50  0001 C CNN "JLCPCB_CORRECTION"
 	1    14950 2750
 	-1   0    0    1
@@
 F 3 "~" H 14950 3150 50  0001 C CNN
 F 4 "C49257" H 14922 3173 50  0001 C CNN "LCSC"
-F 5 "2.54;0;-90" H 14922 3173 50  0001 C CNN "JLCPCB_CORRECTION"
+F 5 "0;2.54;-90" H 14922 3173 50  0001 C CNN "JLCPCB_CORRECTION"
 	1    14950 3150
 	-1   0    0    1
@@
 F 3 "~" H 14950 3550 50  0001 C CNN
 F 4 "C49257" H 14922 3573 50  0001 C CNN "LCSC"
-F 5 "2.54;0;-90" H 14922 3573 50  0001 C CNN "JLCPCB_CORRECTION"
+F 5 "0;2.54;-90" H 14922 3573 50  0001 C CNN "JLCPCB_CORRECTION"
 	1    14950 3550
 	-1   0    0    1
@@
 F 3 "~" H 7250 2700 50  0001 C CNN
 F 4 "C157991" H 7222 2723 50  0001 C CNN "LCSC"
-F 5 "-5;0;-90" H 7222 2723 50  0001 C CNN "JLCPCB_CORRECTION"
+F 5 "-5;0;-180" H 7222 2723 50  0001 C CNN "JLCPCB_CORRECTION"
 	1    7250 2700
 	-1   0    0    -1
@@
 F 3 "~" H 8650 2700 50  0001 C CNN
 F 4 "C157991" H 8622 2723 50  0001 C CNN "LCSC"
-F 5 "-5;0;-90" H 8622 2723 50  0001 C CNN "JLCPCB_CORRECTION"
+F 5 "-5;0;-180" H 8622 2723 50  0001 C CNN "JLCPCB_CORRECTION"
 	1    8650 2700
 	-1   0    0    -1
@@
 F 3 "~" H 14950 3950 50  0001 C CNN
 F 4 "C49257" H 14922 3973 50  0001 C CNN "LCSC"
-F 5 "2.54;0;-90" H 14922 3973 50  0001 C CNN "JLCPCB_CORRECTION"
+F 5 "0;2.54;-90" H 14922 3973 50  0001 C CNN "JLCPCB_CORRECTION"
 	1    14950 3950
 	-1   0    0    1
@@
 F 3 "~" H 14950 4350 50  0001 C CNN
 F 4 "C49257" H 14922 4373 50  0001 C CNN "LCSC"
-F 5 "2.54;0;-90" H 14922 4373 50  0001 C CNN "JLCPCB_CORRECTION"
+F 5 "0;2.54;-90" H 14922 4373 50  0001 C CNN "JLCPCB_CORRECTION"
 	1    14950 4350
 	-1   0    0    1
@@
 F 4 "C8465" H 1600 900 50  0001 C CNN "LCSC"
 F 5 "C395868" H 1600 900 50  0001 C CNN "LCSC_ALT_SCREW_DIBO"
-F 6 "-2.40;0;180" H 1600 900 50  0001 C CNN "JLCPCB_CORRECTION"
+F 6 "2.40;0;180" H 1600 900 50  0001 C CNN "JLCPCB_CORRECTION"
 	1    1600 900
 	1    0    0    -1
@@
 F 4 "C8465" H 1600 1100 50  0001 C CNN "LCSC"
 F 5 "C395868" H 1600 1100 50  0001 C CNN "LCSC_ALT_SCREW_DIBO"
-F 6 "-2.40;0;180" H 1600 1100 50  0001 C CNN "JLCPCB_CORRECTION"
+F 6 "2.40;0;180" H 1600 1100 50  0001 C CNN "JLCPCB_CORRECTION"
 	1    1600 1100
 	1    0    0    -1
@@
 F 4 "C8465" H 1600 1300 50  0001 C CNN "LCSC"
 F 5 "C395868" H 1600 1300 50  0001 C CNN "LCSC_ALT_SCREW_DIBO"
-F 6 "-2.40;0;180" H 1600 1300 50  0001 C CNN "JLCPCB_CORRECTION"
+F 6 "2.40;0;180" H 1600 1300 50  0001 C CNN "JLCPCB_CORRECTION"
 	1    1600 1300
 	1    0    0    -1

Commit message: More placement adjustments
Parts:
- J12, J13, J3, J5, J6, J7: JLCPCB_CORRECTION -5;0;-180 -> 5;0;-180
- J16, J17, J18: JLCPCB_CORRECTION 2.40;0;180 -> 2.54;0;180
Changed lines of the file:
@@
 F 3 "~" H 1700 2700 50  0001 C CNN
 F 4 "C157991" H 1672 2723 50  0001 C CNN "LCSC"
-F 5 "-5;0;-180" H 1672 2723 50  0001 C CNN "JLCPCB_CORRECTION"
+F 5 "5;0;-180" H 1672 2723 50  0001 C CNN "JLCPCB_CORRECTION"
 	1    1700 2700
 	-1   0    0    -1
@@
 F 3 "~" H 3100 2700 50  0001 C CNN
 F 4 "C157991" H 3072 2723 50  0001 C CNN "LCSC"
-F 5 "-5;0;-180" H 3072 2723 50  0001 C CNN "JLCPCB_CORRECTION"
+F 5 "5;0;-180" H 3072 2723 50  0001 C CNN "JLCPCB_CORRECTION"
 	1    3100 2700
 	-1   0    0    -1
@@
 F 3 "~" H 4500 2700 50  0001 C CNN
 F 4 "C157991" H 4472 2723 50  0001 C CNN "LCSC"
-F 5 "-5;0;-180" H 4472 2723 50  0001 C CNN "JLCPCB_CORRECTION"
+F 5 "5;0;-180" H 4472 2723 50  0001 C CNN "JLCPCB_CORRECTION"
 	1    4500 2700
 	-1   0    0    -1
@@
 F 3 "~" H 5900 2700 50  0001 C CNN
 F 4 "C157991" H 5872 2723 50  0001 C CNN "LCSC"
-F 5 "-5;0;-180" H 5872 2723 50  0001 C CNN "JLCPCB_CORRECTION"
+F 5 "5;0;-180" H 5872 2723 50  0001 C CNN "JLCPCB_CORRECTION"
 	1    5900 2700
 	-1   0    0    -1
@@
 F 3 "~" H 7250 2700 50  0001 C CNN
 F 4 "C157991" H 7222 2723 50  0001 C CNN "LCSC"
-F 5 "-5;0;-180" H 7222 2723 50  0001 C CNN "JLCPCB_CORRECTION"
+F 5 "5;0;-180" H 7222 2723 50  0001 C CNN "JLCPCB_CORRECTION"
 	1    7250 2700
 	-1   0    0    -1
@@
 F 3 "~" H 8650 2700 50  0001 C CNN
 F 4 "C157991" H 8622 2723 50  0001 C CNN "LCSC"
-F 5 "-5;0;-180" H 8622 2723 50  0001 C CNN "JLCPCB_CORRECTION"
+F 5 "5;0;-180" H 8622 2723 50  0001 C CNN "JLCPCB_CORRECTION"
 	1    8650 2700
 	-1   0    0    -1
@@
 F 4 "C8465" H 1600 900 50  0001 C CNN "LCSC"
 F 5 "C395868" H 1600 900 50  0001 C CNN "LCSC_ALT_SCREW_DIBO"
-F 6 "2.40;0;180" H 1600 900 50  0001 C CNN "JLCPCB_CORRECTION"
+F 6 "2.54;0;180" H 1600 900 50  0001 C CNN "JLCPCB_CORRECTION"
 	1    1600 900
 	1    0    0    -1
@@
 F 4 "C8465" H 1600 1100 50  0001 C CNN "LCSC"
 F 5 "C395868" H 1600 1100 50  0001 C CNN "LCSC_ALT_SCREW_DIBO"
-F 6 "2.40;0;180" H 1600 1100 50  0001 C CNN "JLCPCB_CORRECTION"
+F 6 "2.54;0;180" H 1600 1100 50  0001 C CNN "JLCPCB_CORRECTION"
 	1    1600 1100
 	1    0    0    -1
@@
 F 4 "C8465" H 1600 1300 50  0001 C CNN "LCSC"
 F 5 "C395868" H 1600 1300 50  0001 C CNN "LCSC_ALT_SCREW_DIBO"
-F 6 "2.40;0;180" H 1600 1300 50  0001 C CNN "JLCPCB_CORRECTION"
+F 6 "2.54;0;180" H 1600 1300 50  0001 C CNN "JLCPCB_CORRECTION"
 	1    1600 1300
 	1    0    0    -1
